Commit message: Added blank macro element to dimensions

File: hros1_description/urdf/hros1_dimensions.xacro (robot description, xacro)
@@ -1 +1,3 @@
 <?xml version="1.0"?>
+<xacro:macro name="blank">
+</xacro:macro>

Commit message: Added robot tag to dimensions file

File: hros1_description/urdf/hros1_dimensions.xacro (robot description, xacro)
@@ -1,4 +1,6 @@
 <?xml version="1.0"?>
-<xacro:macro name="blank">
-<!-- Blank -->
-</xacro:macro>
+<robot xmlns:xacro="http://ros.org/wiki/xacro">
+    <xacro:macro name="blank">
+    <!-- Blank -->
+    </xacro:macro>
+</robot>
