Commit message: Made changes to neck file. Committing to check

File: hros1_description/urdf/hros1_neck.xacro (robot description, xacro)
@@ -5,19 +5,16 @@
     <!--  ATTACHED TO TOP OF BODY -->
     <link name='HR-OS1::neck_link_1_link'>
-      <pose>0 0 0 0 -0 0</pose>
+      <origin xyz="0 0 0" rpy="0 -0 0"/>
       <gravity>1</gravity>
       <self_collide>0</self_collide>
       <kinematic>0</kinematic>
       <visual name='neck_link_1_visual'>
-        <pose>0 0 0 0 -0 0</pose>
+        <origin xyz="0 0 0 0 -0 0"/>
         <geometry>
-          <mesh>
-            <uri>model://HR-OS1/meshes/HROS1_Simple - Neck_Link_1.stl</uri>
-            <scale>1 1 1</scale>
-          </mesh>
+          <mesh filename="package://hros1_description/meshes/HROS1_Simple - Neck_Link_1.stl"/>
         </geometry>
         <material>
           <script>
-            <uri>file://media/materials/scripts/gazebo.material</uri>
+            <uri>file://media/materials/scripts/gazebo.material"
             <name>Gazebo/Grey</name>
           </script>
@@ -25,5 +22,5 @@
       </visual>
       <inertial>
-        <pose>0 -0.101 0.208 0 -0 0</pose>
+        <origin xyz="0 -0.101 0.208 0 -0 0"/>
         <mass>0.005</mass>
         <inertia>
@@ -45,5 +42,5 @@
       <xyz>0 0 1</xyz>
     </axis>
-    <pose>0 -0.045 0 0 0 0</pose>
+    <origin xyz="0 -0.045 0" rpy="0 0 0"/>
   </joint>
   <joint name="neck_base_platform_free_joint" type="revolute">
@@ -53,5 +50,5 @@
       <xyz>1 0 0</xyz>
     </axis>
-    <pose>0 -0.046 0.2 0 0 0</pose>
+    <origin xyz="0 -0.046 0.2" rpy="0 0 0"/>
   </joint>
   <joint name="neck_pitch_1_free_joint" type="revolute">
@@ -61,5 +58,5 @@
       <xyz>1 0 0</xyz>
     </axis>
-    <pose>0 -0.105 0.19 0 0 0</pose>
+    <origin xyz="0 -0.105 0.19" rpy="0 0 0"/>
   </joint>
   <joint name="neck_pitch_2_free_joint" type="revolute">
@@ -69,5 +66,5 @@
       <xyz>1 0 0</xyz>
     </axis>
-    <pose>0 -0.105 0.23 0 0 0</pose>
+    <origin xyz="0 -0.105 0.23" rpy="0 0 0"/>
   </joint>
   <joint name="neck_pitch_main_powered_joint" type="revolute">
@@ -77,5 +74,5 @@
       <xyz>-1 0 0</xyz>
     </axis>
-    <pose>0 -0.07 0.23 0 0 0</pose>
+    <origin xyz="0 -0.07 0.23" rpy="0 0 0"/>
   </joint>
 </xacro:macro>

Commit message: Added missing neck links

File: hros1_description/urdf/hros1_neck.xacro (robot description, xacro)
@@ -1,5 +1,127 @@
 <?xml version="1.0"?>
 <robot xmlns:xacro="http://ros.org/wiki/xacro">
-test
+<!--  NECK Head (Pitch Servo) -->
+<!--  ATTACHED TO BACK OF HEAD  -->
+    <link name='HR-OS1::neck_head_link'>
+      <origin xyz="0 0 0" rpy="0 -0 0"/>
+      <gravity>1</gravity>
+      <self_collide>1</self_collide>
+      <kinematic>0</kinematic>
+      <visual name='neck_head_visual'>
+        <origin xyz="0 0 0" rpy="0 -0 0"/>
+        <geometry>
+          <mesh>
+            <uri>model://HR-OS1/meshes/HROS1_Simple - Neck_Head_Servo.stl</uri>
+            <scale>1 1 1</scale>
+          </mesh>
+        </geometry>
+      </visual>
+      <collision name="collision">
+        <origin xyz=" 0.0 -0.05 0.22" rpy="0 0 0 "/>
+        <geometry>
+          <box>
+            <size>0.02 0.02 0.02</size>
+          </box>
+        </geometry>
+      </collision>
+      <inertial>
+        <mass>0.127</mass>
+        <inertia
+          ixx="0.000036"
+          ixy="0.00000050"
+          ixz="-0.00000017"
+          iyy="0.000027"
+          iyz="-0.00000037"
+          izz="0.000038"
+          />
+      </inertial>
+    </link>
+<!--  NECK Base (YAW SERVO) -->
+<!--  ATTACHED TO BACK OF HEAD  -->
+    <link name='HR-OS1::neck_base_link'>
+      <origin xyz="0 0 0" rpy="0 -0 0"/>
+      <gravity>1</gravity>
+      <self_collide>0</self_collide>
+      <kinematic>0</kinematic>
+      <visual name='neck_base_visual'>
+        <origin xyz="0 0 0" rpy="0 -0 0"/>
+        <geometry>
+          <mesh filename="model://HR-OS1/meshes/HROS1_Simple - Neck_Base.stl"/>
+        </geometry>
+      </visual>
+      <inertial>
+        <origin xyz="0 -0.068 0.0179" rpy="0 -0 0"/>
+        <mass value="0.075"/>
+        <inertia
+          ixx="0.000029"
+          ixy="0.000000002"
+          ixz="-0.0000000069"
+          iyy="0.000016"
+          iyz="0.00000045"
+          izz="0.000026"
+          />
+      </inertial>
+    </link>
+<!--  Neck Head Platform  -->
+<!--  Supports to head; should be able to tilt  -->
+    <link name='HR-OS1::neck_base_platform_link'>
+      <origin xyz="0 0 0" rpy="0 -0 0"/>
+      <gravity>1</gravity>
+      <self_collide>1</self_collide>
+      <kinematic>0</kinematic>
+      <visual name='neck_base_platform_visual'>
+        <origin xyz="0 0 0" rpy="0 -0 0"/>
+        <geometry>
+          <mesh filename="package://hros1_description/meshes/HROS1_Simple - Neck_Base_Platform.stl"/>
+        </geometry>
+      </visual>
+      <collision name="collision">
+        <origin xyz="0 -0.046 0.20955" rpy="0 0 0"/>
+        <geometry>
+          <cylinder>
+            <radius>0.02</radius>
+            <length>0.0025</length>
+          </cylinder>
+        </geometry>
+      </collision>
+      <inertial>
+        <origin xyz="0 -0.052 0.207" rpy="0 -0 0"/>
+        <mass value="0.012"/>
+        <inertia
+          ixx="0.0000017"
+          ixy="0.0"
+          ixz="0.0"
+          iyy="0.0000019"
+          iyz="0.0"
+          izz="0.0000034"
+          />
+      </inertial>
+    </link>
+<!--  NECK Link 2  -->
+<!--  ATTACHED TO Head Servo  -->
+    <link name='HR-OS1::neck_link_2_link'>
+      <origin xyz="0 0 0" rpy="0 -0 0"/>
+      <gravity>1</gravity>
+      <self_collide>0</self_collide>
+      <kinematic>0</kinematic>
+      <visual name='neck_link_2_visual'>
+        <origin xyz="0 0 0" rpy="0 -0 0"/>
+        <geometry>
+          <mesh filename="model://HR-OS1/meshes/HROS1_Simple - Neck_Link_2.stl"/>
+        </geometry>
+      </visual>
+      <inertial>
+        <origin xyz="0 -0.077 0.231" rpy="0 -0 0"/>
+        <mass value="0.011"/>
+        <inertia
+          ixx="0.000002"
+          ixy="0.0"
+          ixz="0.0"
+          iyy="0.0000057"
+          iyz="0.0"
+          izz="0.0000071"
+          />
+      </inertial>
+    </link>
 <xacro:macro name="neck_links">
     <!--  ATTACHED TO TOP OF BODY -->

Commit message: Changed collision cylinder in neck

File: hros1_description/urdf/hros1_neck.xacro (robot description, xacro)
@@ -74,8 +74,5 @@
         <origin xyz="0 -0.046 0.20955" rpy="0 0 0"/>
         <geometry>
-          <cylinder>
-            <radius>0.02</radius>
-            <length>0.0025</length>
-          </cylinder>
+          <cylinder radius="0.02" length="0.0025"/>
         </geometry>
       </collision>

Commit message: Fixed inertia tag labels

File: hros1_description/urdf/hros1_neck.xacro (robot description, xacro)
@@ -23,5 +23,5 @@
       </collision>
       <inertial>
-        <mass>0.127</mass>
+        <mass value="0.127"/>
         <inertia
           ixx="0.000036"

File: hros1_description/urdf/hros1_right_leg.xacro (robot description, xacro)
@@ -19,5 +19,5 @@
         <inertia
           ixx="0.000016"
-          <ixy="0.0"
+          ixy="0.0"
           ixz="0.0"
           iyy="0.0000035"
@@ -44,5 +44,5 @@
         <inertia
           ixx="0.000058"
-          <ixy="0.00000045"
+          ixy="0.00000045"
           ixz="0.00000027"
           iyy="0.000029"
@@ -69,5 +69,5 @@
         <inertia
           ixx="0.000016"
-          <ixy="0.0"
+          ixy="0.0"
           ixz="0.0"
           iyy="0.000023"
@@ -94,5 +94,5 @@
         <inertia
           ixx="0.000013"
-          <ixy="0.00000025"
+          ixy="0.00000025"
           ixz="0.000000071"
           iyy="0.0000090"
@@ -119,5 +119,5 @@
         <inertia
           ixx="0.0000094"
-          <ixy="0.0"
+          ixy="0.0"
           ixz="0.0"
           iyy="0.000014"
@@ -144,5 +144,5 @@
         <inertia
           ixx="0.000058"
-          <ixy="0.00000051"
+          ixy="0.00000051"
           ixz="-0.00000024"
           iyy="0.000029"
@@ -177,5 +177,5 @@
         <inertia
           ixx="0.00006"
-          <ixy="-0.0000017"
+          ixy="-0.0000017"
           ixz="-0.0000011"
           iyy="0.000026"

Commit message: Changed neck link visual file reference

File: hros1_description/urdf/hros1_neck.xacro (robot description, xacro)
@@ -100,5 +100,5 @@
         <origin xyz="0 0 0" rpy="0 -0 0"/>
         <geometry>
-          <mesh filename="model://HR-OS1/meshes/HROS1_Simple - Neck_Link_2.stl"/>
+          <mesh filename="package://hros1_description/meshes/HROS1_Simple - Neck_Link_2.stl"/>
         </geometry>
       </visual>

Commit message: Made changes to neck file

File: hros1_description/urdf/hros1_neck.xacro (robot description, xacro)
@@ -11,5 +11,5 @@
         <origin xyz="0 0 0" rpy="0 -0 0"/>
         <geometry>
-          <mesh filename="model://HR-OS1/meshes/HROS1_Simple - Neck_Head_Servo.stl"/>
+          <mesh filename="package://hros1_description/meshes/HROS1_Simple - Neck_Head_Servo.stl"/>
         </geometry>
       </visual>
@@ -42,5 +42,5 @@
         <origin xyz="0 0 0" rpy="0 -0 0"/>
         <geometry>
-          <mesh filename="model://HR-OS1/meshes/HROS1_Simple - Neck_Base.stl"/>
+          <mesh filename="package://hros1_description/meshes/HROS1_Simple - Neck_Base.stl"/>
         </geometry>
       </visual>

Commit message: Changed reference to moved visuals

File: hros1_description/urdf/hros1_neck.xacro (robot description, xacro)
@@ -11,5 +11,5 @@
         <origin xyz="0 0 0" rpy="0 -0 0"/>
         <geometry>
-          <mesh filename="package://hros1_description/meshes/HROS1_Simple - Neck_Head_Servo.stl"/>
+          <mesh filename="package://hros1_description/meshes/hros1_neck_head_servo_moved.stl"/>
         </geometry>
       </visual>
@@ -35,16 +35,16 @@
 <!--  ATTACHED TO BACK OF HEAD  -->
     <link name='neck_base_link'>
-      <origin xyz="0 0 0" rpy="0 -0 0"/>
+      <!--<origin xyz="0 0.18 0.188" rpy="0 -0 0"/>-->
       <gravity>1</gravity>
       <self_collide>0</self_collide>
       <kinematic>0</kinematic>
       <visual name='neck_base_visual'>
-        <origin xyz="0 0 0" rpy="0 -0 0"/>
+        <origin xyz="0 0.052 0" rpy="0 -0 0"/>
         <geometry>
-          <mesh filename="package://hros1_description/meshes/HROS1_Simple - Neck_Base.stl"/>
+          <mesh filename="package://hros1_description/meshes/hros1_neck_base_moved.stl"/>
         </geometry>
       </visual>
       <inertial>
-        <origin xyz="0 -0.068 0.0179" rpy="0 -0 0"/>
+        <origin xyz="0 0.052 0" rpy="0 -0 0"/>
         <mass value="0.075"/>
         <inertia
@@ -66,7 +66,7 @@
       <kinematic>0</kinematic>
       <visual name='neck_base_platform_visual'>
-        <origin xyz="0 0 0" rpy="0 -0 0"/>
+        <origin xyz="0 0.98 -.20" rpy="0 -0 0"/>
         <geometry>
-          <mesh filename="package://hros1_description/meshes/HROS1_Simple - Neck_Base_Platform.stl"/>
+          <mesh filename="package://hros1_description/meshes/hros1_neck_base_platform_moved.stl"/>
         </geometry>
       </visual>
@@ -100,5 +100,5 @@
         <origin xyz="0 0 0" rpy="0 -0 0"/>
         <geometry>
-          <mesh filename="package://hros1_description/meshes/HROS1_Simple - Neck_Link_2.stl"/>
+          <mesh filename="package://hros1_description/meshes/hros1_neck_link_2_moved.stl"/>
         </geometry>
       </visual>
@@ -126,5 +126,5 @@
         <origin xyz="0 0 0" rpy="0 -0 0"/>
         <geometry>
-          <mesh filename="package://hros1_description/meshes/HROS1_Simple - Neck_Link_1.stl"/>
+          <mesh filename="package://hros1_description/meshes/hros1_neck_link_2_moved.stl"/>
         </geometry>
       </visual>
@@ -151,5 +151,5 @@
       <xyz>0 0 1</xyz>
     </axis>
-    <origin xyz="0 -0.045 0" rpy="0 0 0"/>
+    <origin xyz="0 -0.052 0" rpy="0 0 0"/>
   </joint>
   <joint name="neck_base_platform_free_joint" type="continuous">

File: hros1_description/urdf/hros1_robot.urdf.xacro (robot description, xacro)
@@ -4,12 +4,15 @@
     <xacro:include filename="$(find hros1_description)/urdf/hros1_body.xacro"/>
     <xacro:include filename="$(find hros1_description)/urdf/hros1_neck.xacro"/>
+<!--
     <xacro:include filename="$(find hros1_description)/urdf/hros1_left_arm.xacro"/>
     <xacro:include filename="$(find hros1_description)/urdf/hros1_left_leg.xacro"/>
     <xacro:include filename="$(find hros1_description)/urdf/hros1_right_arm.xacro"/>
     <xacro:include filename="$(find hros1_description)/urdf/hros1_right_leg.xacro"/>
+  -->
     <xacro:body_links />
     <xacro:body_joints />
     <xacro:neck_links />
     <xacro:neck_joints />
+    <!--
     <xacro:left_arm_links />
     <xacro:left_arm_joints />
@@ -20,3 +23,4 @@
     <xacro:right_leg_links />
     <xacro:right_leg_joints />
+    -->
 </robot>

Commit message: Got neck working

File: hros1_description/urdf/hros1_neck.xacro (robot description, xacro)
@@ -40,5 +40,6 @@
       <kinematic>0</kinematic>
       <visual name='neck_base_visual'>
-        <origin xyz="0 0.052 0" rpy="0 -0 0"/>
+        <origin xyz="0 0 0" rpy="0 0 0"/>
+        <!--<origin xyz="0 0.052 0" rpy="0 -0 0"/>-->
         <geometry>
           <mesh filename="package://hros1_description/meshes/hros1_neck_base_moved.stl"/>
@@ -66,5 +67,6 @@
       <kinematic>0</kinematic>
       <visual name='neck_base_platform_visual'>
-        <origin xyz="0 0.98 -.20" rpy="0 -0 0"/>
+        <origin xyz="0 0 0" rpy="0 0 0"/>
+        <!--<origin xyz="0 0.98 -.20" rpy="0 -0 0"/>-->
         <geometry>
           <mesh filename="package://hros1_description/meshes/hros1_neck_base_platform_moved.stl"/>
@@ -126,5 +128,5 @@
         <origin xyz="0 0 0" rpy="0 -0 0"/>
         <geometry>
-          <mesh filename="package://hros1_description/meshes/hros1_neck_link_2_moved.stl"/>
+          <mesh filename="package://hros1_description/meshes/hros1_neck_link_1_moved.stl"/>
         </geometry>
       </visual>
@@ -151,5 +153,5 @@
       <xyz>0 0 1</xyz>
     </axis>
-    <origin xyz="0 -0.052 0" rpy="0 0 0"/>
+    <origin xyz="0 -0.052 0.162" rpy="0 0 3.1415"/>
   </joint>
   <joint name="neck_base_platform_free_joint" type="continuous">
@@ -160,5 +162,5 @@
       <xyz>1 0 0</xyz>
     </axis>
-    <origin xyz="0 -0.046 0.2" rpy="0 0 0"/>
+    <origin xyz="0 0 0.042" rpy="0 0 0"/>
   </joint>
   <joint name="neck_pitch_1_free_joint" type="continuous">
@@ -169,5 +171,5 @@
       <xyz>1 0 0</xyz>
     </axis>
-    <origin xyz="0 -0.105 0.19" rpy="0 0 0"/>
+    <origin xyz="0 0.049 0.026" rpy="0 0 0"/>
   </joint>
   <joint name="neck_pitch_2_free_joint" type="continuous">
@@ -178,5 +180,5 @@
       <xyz>1 0 0</xyz>
     </axis>
-    <origin xyz="0 -0.105 0.23" rpy="0 0 0"/>
+    <origin xyz="0 0 0.048" rpy="0 0 0"/>
   </joint>
   <joint name="neck_pitch_main_powered_joint" type="revolute">
@@ -187,5 +189,5 @@
       <xyz>-1 0 0</xyz>
     </axis>
-    <origin xyz="0 -0.07 0.23" rpy="0 0 0"/>
+    <origin xyz="0 -0.034 0.0" rpy="0 0 0"/>
   </joint>
 </xacro:macro>
