Commit message: Added test meshes for moved components

File: hros1_description/urdf/hros1_left_leg.xacro (robot description, xacro)
@@ -221,13 +221,9 @@
     <limit effort="1" velocity="1" upper="3.1415" lower="-3.1415"/>
   </joint>
-  <joint name="left_knee-shin_fixed_joint" type="revolute">
+  <joint name="left_knee-shin_fixed_joint" type="fixed">
     <parent link="left_leg_knee_link"/>
     <child link="left_leg_shin_link"/>
     <axis>
       <xyz>1 0 0</xyz>
-      <limit>
-          <lower>0</lower>
-          <upper>0</upper>
-      </limit>
     </axis>
     <origin xyz="-0.015 -0.04 -0.09" rpy="0 0 0"/>

Commit message: Changed positioning of links/joints to get left leg working

File: hros1_description/urdf/hros1_left_leg.xacro (robot description, xacro)
@@ -11,5 +11,5 @@
         <origin xyz="0 0 0" rpy="0 -0 0"/>
         <geometry>
-          <mesh filename="package://hros1_description/meshes/HROS1_Simple - Left_Leg_Yaw_Link.stl"/>
+          <mesh filename="package://hros1_description/meshes/hros1_left_leg_yaw_link_moved.stl"/>
         </geometry>
       </visual>
@@ -28,5 +28,4 @@
     </link>
 <!-- LEFT LOWER HIP  -->
-<!--
     <link name='left_leg_lower_hip_link'>
       <origin xyz="0 0 0 0 -0 0"/>
@@ -37,5 +36,5 @@
         <origin xyz="0 0 0" rpy="0 -0 0"/>
         <geometry>
-          <mesh filename="package://hros1_description/meshes/HROS1_Simple - Left_Leg_Hip_Joint.stl"/>
+          <mesh filename="package://hros1_description/meshes/hros1_left_leg_hip_joint_moved.stl"/>
         </geometry>
       </visual>
@@ -53,7 +52,5 @@
       </inertial>
     </link>
--->
 <!-- LEFT THIGH  -->
-<!--
     <link name='left_leg_thigh_link'>
       <origin xyz="0 0 0 0 -0 0"/>
@@ -64,5 +61,5 @@
         <origin xyz="0 0 0" rpy="0 -0 0"/>
         <geometry>
-          <mesh filename="package://hros1_description/meshes/HROS1_Simple - Left_Leg_Thigh.stl"/>
+          <mesh filename="package://hros1_description/meshes/hros1_left_leg_thigh_moved.stl"/>
         </geometry>
       </visual>
@@ -80,7 +77,5 @@
       </inertial>
     </link>
--->
 <!-- LEFT KNEE  -->
-<!--
     <link name='left_leg_knee_link'>
       <origin xyz="0 0 0" rpy="0 -0 0"/>
@@ -91,5 +86,5 @@
         <origin xyz="0 0 0" rpy="0 -0 0"/>
         <geometry>
-          <mesh filename="package://hros1_description/meshes/HROS1_Simple - Left_Leg_Knee.stl"/>
+          <mesh filename="package://hros1_description/meshes/hros1_left_leg_knee_moved.stl"/>
         </geometry>
       </visual>
@@ -107,7 +102,5 @@
       </inertial>
     </link>
--->
 <!-- LEFT SHIN  -->
-<!--
     <link name='left_leg_shin_link'>
       <origin xyz="0 0 0" rpy="0 -0 0"/>
@@ -118,5 +111,5 @@
         <origin xyz="0 0 0" rpy="0 -0 0"/>
         <geometry>
-          <mesh filename="package://hros1_description/meshes/HROS1_Simple - Left_Leg_Shin.stl"/>
+          <mesh filename="package://hros1_description/meshes/hros1_left_leg_shin_moved.stl"/>
         </geometry>
       </visual>
@@ -134,7 +127,5 @@
       </inertial>
     </link>
--->
 <!-- LEFT ANKLE  -->
-<!--
     <link name='left_leg_ankle_link'>
       <origin xyz="0 0 0" rpy="0 -0 0"/>
@@ -145,5 +136,5 @@
         <origin xyz="0 0 0" rpy="0 -0 0"/>
         <geometry>
-          <mesh filename="package://hros1_description/meshes/HROS1_Simple - Left_Leg_Ankle_Joint.stl"/>
+          <mesh filename="package://hros1_description/meshes/hros1_left_leg_ankle_joint_moved.stl"/>
         </geometry>
       </visual>
@@ -161,7 +152,5 @@
       </inertial>
     </link>
--->
 <!-- LEFT FOOT  -->
-<!--
     <link name='left_leg_foot_link'>
       <origin xyz="0 0 0" rpy="0 -0 0"/>
@@ -172,5 +161,5 @@
         <origin xyz="0 0 0" rpy="0 -0 0"/>
         <geometry>
-          <mesh filename="package://hros1_description/meshes/HROS1_Simple - Left_Leg_Foot.stl"/>
+          <mesh filename="package://hros1_description/meshes/hros1_left_leg_foot_moved.stl"/>
         </geometry>
       </visual>
@@ -201,13 +190,12 @@
     <child link="left_leg_upper_hip_link"/>
     <axis xyz="0 0 1"/>
-    <origin xyz="-0.040 -0.045 0" rpy="0 0 0"/>
-    <limit effort="1" velocity="1" upper="3.1415" lower="-3.1415"/>
-  </joint>
-  <!--
+    <origin xyz="0.039 0.045 0.023" rpy="0 0 0"/>
+    <limit effort="1" velocity="1" upper="3.1415" lower="-3.1415"/>
+  </joint>
   <joint name="left_hip_roll_powered_joint" type="revolute">
     <parent link="left_leg_upper_hip_link"/>
     <child link="left_leg_lower_hip_link"/>
-    <axis xyz="0 0 1"/>
-    <origin xyz="-0.040 -0.045 -0.01" rpy="0 0 0"/>
+    <axis xyz="0 1 0"/>
+    <origin xyz="0 0.053 -0.036" rpy="0 0 0"/>
     <limit effort="1" velocity="1" upper="3.1415" lower="-3.1415"/>
   </joint>
@@ -215,6 +203,6 @@
     <parent link="left_leg_lower_hip_link"/>
     <child link="left_leg_thigh_link"/>
-    <axis xyz="0 0 1"/>
-    <origin xyz="-0.040 -0.045 -0.01" rpy="0 0 0"/>
+    <axis xyz="1 0 0"/>
+    <origin xyz="-0.015 -0.053 0" rpy="0 0 0"/>
     <limit effort="1" velocity="1" upper="3.1415" lower="-3.1415"/>
   </joint>
@@ -222,6 +210,6 @@
     <parent link="left_leg_thigh_link"/>
     <child link="left_leg_knee_link"/>
-    <axis xyz="0 0 1"/>
-    <origin xyz="-0.015 -0.04 -0.09" rpy="0 0 0"/>
+    <axis xyz="1 0 0"/>
+    <origin xyz="-0.006 -0.006 -0.077" rpy="0 0 0"/>
     <limit effort="1" velocity="1" upper="3.1415" lower="-3.1415"/>
   </joint>
@@ -230,5 +218,5 @@
     <child link="left_leg_shin_link"/>
     <axis xyz="0 0 1"/>
-    <origin xyz="-0.015 -0.04 -0.09" rpy="0 0 0"/>
+    <origin xyz="0.004 -0.002 -0.015" rpy="0 0 0"/>
     <limit effort="1" velocity="1" upper="3.1415" lower="-3.1415"/>
   </joint>
@@ -236,6 +224,6 @@
     <parent link="left_leg_shin_link"/>
     <child link="left_leg_ankle_link"/>
-    <axis xyz="0 0 1"/>
-    <origin xyz="-0.015 -0.045 -0.16" rpy="0 0 0"/>
+    <axis xyz="1 0 0"/>
+    <origin xyz="-0.004 0.008 -0.058" rpy="0 0 0"/>
     <limit effort="1" velocity="1" upper="3.1415" lower="-3.1415"/>
   </joint>
@@ -243,9 +231,8 @@
     <parent link="left_leg_ankle_link"/>
     <child link="left_leg_foot_link"/>
-    <axis xyz="0 0 1"/>
-    <origin xyz="-0.04 -0.045 -0.16" rpy="0 0 0"/>
-    <limit effort="1" velocity="1" upper="3.1415" lower="-3.1415"/>
-  </joint>
-  -->
+    <axis xyz="0 1 0"/>
+    <origin xyz="0.021 0.053 0" rpy="0 0 0"/>
+    <limit effort="1" velocity="1" upper="3.1415" lower="-3.1415"/>
+  </joint>
 </xacro:macro>
 </robot>

File: hros1_description/urdf/hros1_robot.urdf (robot description, URDF)
Before this commit: robot hros1, 14 links, 13 joints
Links:
- added link left_leg_ankle_link, mass 0.110; visual mesh filename=package://hros1_description/meshes/hros1_left_leg_ankle_joi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
- added link left_leg_foot_link, mass 0.067; collision box size=0.065 .1 0.01; visual mesh filename=package://hros1_description/meshes/hros1_left_leg_foot_move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
- added link left_leg_knee_link, mass 0.055; visual mesh filename=package://hros1_description/meshes/hros1_left_leg_knee_move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
- added link left_leg_lower_hip_link, mass 0.110; visual mesh filename=package://hros1_description/meshes/hros1_left_leg_hip_joint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
- added link left_leg_shin_link, mass 0.021; visual mesh filename=package://hros1_description/meshes/hros1_left_leg_shin_move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
- added link left_leg_thigh_link, mass 0.028; visual mesh filename=package://hros1_description/meshes/hros1_left_leg_thigh_mov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
- link left_leg_upper_hip_link: geometry visual mesh filename=package://hros1_description/meshes/hros1_left_leg_yaw_link_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
Joints:
- added joint left_ankle_pitch_powered_joint: type revolute, parent left_leg_shin_link, child left_leg_ankle_link, origin xyz=-0.004 0.008 -0.058 rpy=0 0 0, axis 1 0 0, limit lower=-3.1415 upper=3.1415 effort=1 velocity=1
- added joint left_ankle_roll_powered_joint: type revolute, parent left_leg_ankle_link, child left_leg_foot_link, origin xyz=0.021 0.053 0 rpy=0 0 0, axis 0 1 0, limit lower=-3.1415 upper=3.1415 effort=1 velocity=1
- added joint left_hip_pitch_powered_joint: type revolute, parent left_leg_lower_hip_link, child left_leg_thigh_link, origin xyz=-0.015 -0.053 0 rpy=0 0 0, axis 1 0 0, limit lower=-3.1415 upper=3.1415 effort=1 velocity=1
- added joint left_hip_roll_powered_joint: type revolute, parent left_leg_upper_hip_link, child left_leg_lower_hip_link, origin xyz=0 0.053 -0.036 rpy=0 0 0, axis 0 1 0, limit lower=-3.1415 upper=3.1415 effort=1 velocity=1
- added joint left_knee-shin_fixed_joint: type fixed, parent left_leg_knee_link, child left_leg_shin_link, origin xyz=0.004 -0.002 -0.015 rpy=0 0 0, axis 0 0 1, limit lower=-3.1415 upper=3.1415 effort=1 velocity=1
- added joint left_knee_pitch_powered_joint: type revolute, parent left_leg_thigh_link, child left_leg_knee_link, origin xyz=-0.006 -0.006 -0.077 rpy=0 0 0, axis 1 0 0, limit lower=-3.1415 upper=3.1415 effort=1 velocity=1
- joint left_hip_yaw_powered_joint: origin xyz=-0.040 -0.045 0 rpy=0 0 0 -> xyz=0.039 0.045 0.023 rpy=0 0 0
