Commit message: Got correct mesh files in model, and arranged parts correctly

File: hros1_description/urdf/hros1_left_arm.xacro (robot description, xacro)
@@ -11,5 +11,5 @@
             <origin xyz="0 0 0" rpy="0 -0 0"/>
             <geometry>
-              <mesh filename="package://hros1_description/meshes/hros1_left_arm_shoulder_moved.stl"/>
+              <mesh filename="package://hros1_description/meshes/left_arm_shoulder.stl"/>
             </geometry>
           </visual>
@@ -36,5 +36,5 @@
             <origin xyz="0 0 0" rpy="0 -0 0"/>
             <geometry>
-              <mesh filename="package://hros1_description/meshes/hros1_left_arm_upper_servo_moved.stl"/>
+              <mesh filename="package://hros1_description/meshes/left_arm_upper_servo.stl"/>
             </geometry>
           </visual>
@@ -61,5 +61,5 @@
             <origin xyz="0 0 0" rpy="0 -0 0"/>
             <geometry>
-              <mesh filename="package://hros1_description/meshes/hros1_left_arm_elbow_link_moved.stl"/>
+              <mesh filename="package://hros1_description/meshes/left_arm_elbow_link.stl"/>
             </geometry>
           </visual>
@@ -86,5 +86,5 @@
             <origin xyz="0 0 0" rpy="0 -0 0"/>
             <geometry>
-              <mesh filename="package://hros1_description/meshes/hros1_left_arm_forearm_servo_moved.stl"/>
+              <mesh filename="package://hros1_description/meshes/left_arm_forearm_servo.stl"/>
             </geometry>
           </visual>

File: hros1_description/urdf/hros1_left_leg.xacro (robot description, xacro)
@@ -11,5 +11,5 @@
         <origin xyz="0 0 0" rpy="0 -0 0"/>
         <geometry>
-          <mesh filename="package://hros1_description/meshes/hros1_left_leg_yaw_link_moved.stl"/>
+          <mesh filename="package://hros1_description/meshes/left_leg_yaw_link.stl"/>
         </geometry>
       </visual>
@@ -36,5 +36,5 @@
         <origin xyz="0 0 0" rpy="0 -0 0"/>
         <geometry>
-          <mesh filename="package://hros1_description/meshes/hros1_left_leg_hip_joint_moved.stl"/>
+          <mesh filename="package://hros1_description/meshes/left_leg_hip_joint.stl"/>
         </geometry>
       </visual>
@@ -61,5 +61,5 @@
         <origin xyz="0 0 0" rpy="0 -0 0"/>
         <geometry>
-          <mesh filename="package://hros1_description/meshes/hros1_left_leg_thigh_moved.stl"/>
+          <mesh filename="package://hros1_description/meshes/left_leg_thigh.stl"/>
         </geometry>
       </visual>
@@ -86,5 +86,5 @@
         <origin xyz="0 0 0" rpy="0 -0 0"/>
         <geometry>
-          <mesh filename="package://hros1_description/meshes/hros1_left_leg_knee_moved.stl"/>
+          <mesh filename="package://hros1_description/meshes/left_leg_knee.stl"/>
         </geometry>
       </visual>
@@ -111,5 +111,5 @@
         <origin xyz="0 0 0" rpy="0 -0 0"/>
         <geometry>
-          <mesh filename="package://hros1_description/meshes/hros1_left_leg_shin_moved.stl"/>
+          <mesh filename="package://hros1_description/meshes/left_leg_shin.stl"/>
         </geometry>
       </visual>
@@ -136,5 +136,5 @@
         <origin xyz="0 0 0" rpy="0 -0 0"/>
         <geometry>
-          <mesh filename="package://hros1_description/meshes/hros1_left_leg_ankle_joint_moved.stl"/>
+          <mesh filename="package://hros1_description/meshes/left_leg_ankle_joint.stl"/>
         </geometry>
       </visual>
@@ -161,5 +161,5 @@
         <origin xyz="0 0 0" rpy="0 -0 0"/>
         <geometry>
-          <mesh filename="package://hros1_description/meshes/hros1_left_leg_foot_moved.stl"/>
+          <mesh filename="package://hros1_description/meshes/left_leg_foot.stl"/>
         </geometry>
       </visual>

File: hros1_description/urdf/hros1_neck.xacro (robot description, xacro)
@@ -11,5 +11,5 @@
         <origin xyz="0 0 0" rpy="0 -0 0"/>
         <geometry>
-          <mesh filename="package://hros1_description/meshes/hros1_neck_link_1_moved.stl"/>
+          <mesh filename="package://hros1_description/meshes/neck_link_1.stl"/>
         </geometry>
       </visual>
@@ -37,5 +37,5 @@
         <origin xyz="0 0 0" rpy="0 -0 0"/>
         <geometry>
-          <mesh filename="package://hros1_description/meshes/hros1_neck_head_servo_moved.stl"/>
+          <mesh filename="package://hros1_description/meshes/neck_head_servo.stl"/>
         </geometry>
       </visual>
@@ -68,5 +68,5 @@
         <origin xyz="0 0.0 0" rpy="0 -0 0"/>
         <geometry>
-          <mesh filename="package://hros1_description/meshes/hros1_neck_base_moved.stl"/>
+          <mesh filename="package://hros1_description/meshes/neck_base.stl"/>
         </geometry>
       </visual>
@@ -94,5 +94,5 @@
         <origin xyz="0 0 0" rpy="0 -0 0"/>
         <geometry>
-          <mesh filename="package://hros1_description/meshes/hros1_neck_base_platform_moved.stl"/>
+          <mesh filename="package://hros1_description/meshes/neck_base_platform.stl"/>
         </geometry>
       </visual>
@@ -126,5 +126,5 @@
         <origin xyz="0 0 0" rpy="0 -0 0"/>
         <geometry>
-          <mesh filename="package://hros1_description/meshes/hros1_neck_link_2_moved.stl"/>
+          <mesh filename="package://hros1_description/meshes/neck_link_2.stl"/>
         </geometry>
       </visual>

File: hros1_description/urdf/hros1_right_arm.xacro (robot description, xacro)
@@ -10,5 +10,5 @@
         <origin xyz="0 0 0" rpy="0 -0 0"/>
         <geometry>
-          <mesh filename="package://hros1_description/meshes/HROS1_Simple - Right_Arm_Shoulder.stl"/>
+          <mesh filename="package://hros1_description/meshes/right_arm_shoulder.stl"/>
         </geometry>
       </visual>
@@ -35,5 +35,5 @@
         <origin xyz="0 0 0" rpy="0 -0 0"/>
         <geometry>
-          <mesh filename="package://hros1_description/meshes/HROS1_Simple - Right_Arm_Upper_Servo.stl"/>
+          <mesh filename="package://hros1_description/meshes/right_arm_upper_servo.stl"/>
         </geometry>
       </visual>
@@ -60,5 +60,5 @@
         <origin xyz="0 0 0" rpy="0 -0 0"/>
         <geometry>
-          <mesh filename="package://hros1_description/meshes/HROS1_Simple - Right_Arm_Elbow_Link.stl"/>
+          <mesh filename="package://hros1_description/meshes/right_arm_elbow_link.stl"/>
         </geometry>
       </visual>
@@ -85,5 +85,5 @@
         <origin xyz="0 0 0" rpy="0 -0 0"/>
         <geometry>
-          <mesh filename="package://hros1_description/meshes/HROS1_Simple - Right_Arm_Forearm_Servo.stl"/>
+          <mesh filename="package://hros1_description/meshes/right_arm_forearm_servo.stl"/>
         </geometry>
       </visual>
@@ -106,8 +106,6 @@
     <parent link="body_structure_link"/>
     <child link="right_arm_shoulder_link"/>
-    <axis>
-      <xyz>1 0 0</xyz>
-    </axis>
-    <origin xyz="0 -0.05 0.13" rpy="0 0 0"/>
+    <axis xyz="-1 0 0"/>
+    <origin xyz="-0.051 0.052 0.133" rpy="0 0 0"/>
     <limit effort="1" velocity="1" upper="3.1415" lower="-3.1415"/>
   </joint>
@@ -115,8 +113,6 @@
     <parent link="right_arm_shoulder_link"/>
     <child link="right_arm_upper_servo_link"/>
-    <axis>
-      <xyz>0 -1 0</xyz>
-    </axis>
-    <origin xyz="0.085 -0.05 0.115" rpy="0 0 0"/>
+    <axis xyz="0 -1 0"/>
+    <origin xyz="-0.03 0.02 -0.015" rpy="0 0 0"/>
     <limit effort="1" velocity="1" upper="3.1415" lower="-3.1415"/>
   </joint>
@@ -124,15 +120,12 @@
     <parent link="right_arm_upper_servo_link"/>
     <child link="right_arm_elbow_link"/>
-    <axis>
-      <xyz>0 1 0</xyz>
-    </axis>
+    <axis xyz="0 -1 0"/>
+    <origin xyz="-0.002 -0.033 -0.037" rpy="0 0 0"/>
   </joint>
   <joint name="right_elbow_powered_joint" type="revolute">
     <parent link="right_arm_elbow_link"/>
     <child link="right_arm_forearm_servo_link"/>
-    <axis>
-      <xyz>-1 0 -0.25</xyz>
-    </axis>
-    <origin xyz="0 -0.037 0.03" rpy="0 0 0"/>
+    <axis xyz="-0.8 0.0 -0.2"/>
+    <origin xyz="0.005 0.0 -0.03" rpy="0 0 0"/>
     <limit effort="1" velocity="1" upper="3.1415" lower="-3.1415"/>
   </joint>

File: hros1_description/urdf/hros1_right_leg.xacro (robot description, xacro)
@@ -11,5 +11,5 @@
         <origin xyz="0 0 0" rpy="0 -0 0"/>
         <geometry>
-          <mesh filename="package://hros1_description/meshes/HROS1_Simple - Right_Leg_Yaw_Link.stl"/>
+          <mesh filename="package://hros1_description/meshes/right_leg_yaw_link.stl"/>
         </geometry>
       </visual>
@@ -36,5 +36,5 @@
         <origin xyz="0 0 0" rpy="0 -0 0"/>
         <geometry>
-          <mesh filename="package://hros1_description/meshes/HROS1_Simple - Right_Leg_Hip_Joint.stl"/>
+          <mesh filename="package://hros1_description/meshes/right_leg_hip_joint.stl"/>
         </geometry>
       </visual>
@@ -61,5 +61,5 @@
         <origin xyz="0 0 0" rpy="0 -0 0"/>
         <geometry>
-          <mesh filename="package://hros1_description/meshes/HROS1_Simple - Right_Leg_Thigh.stl"/>
+          <mesh filename="package://hros1_description/meshes/right_leg_thigh.stl"/>
         </geometry>
       </visual>
@@ -86,5 +86,5 @@
         <origin xyz="0 0 0" rpy="0 -0 0"/>
         <geometry>
-          <mesh filename="package://hros1_description/meshes/HROS1_Simple - Right_Leg_Knee.stl"/>
+          <mesh filename="package://hros1_description/meshes/right_leg_knee.stl"/>
         </geometry>
       </visual>
@@ -111,5 +111,5 @@
         <origin xyz="0 0 0" rpy="0 -0 0"/>
         <geometry>
-          <mesh filename="package://hros1_description/meshes/HROS1_Simple - Right_Leg_Shin.stl"/>
+          <mesh filename="package://hros1_description/meshes/right_leg_shin.stl"/>
         </geometry>
       </visual>
@@ -136,5 +136,5 @@
         <origin xyz="0 0 0" rpy="0 -0 0"/>
         <geometry>
-          <mesh filename="package://hros1_description/meshes/HROS1_Simple - Right_Leg_Ankle_Joint.stl"/>
+          <mesh filename="package://hros1_description/meshes/right_leg_ankle_joint.stl"/>
         </geometry>
       </visual>
@@ -161,5 +161,5 @@
         <origin xyz="0 0 0" rpy="0 -0 0"/>
         <geometry>
-          <mesh filename="package://hros1_description/meshes/HROS1_Simple - Right_Leg_Foot.stl"/>
+          <mesh filename="package://hros1_description/meshes/right_leg_foot.stl"/>
         </geometry>
       </visual>
@@ -188,8 +188,6 @@
     <parent link="body_structure_link"/>
     <child link="right_leg_upper_hip_link"/>
-    <axis>
-      <xyz>0 0 -1</xyz>
-    </axis>
-    <origin xyz="0.040 -0.045 0" rpy="0 0 0"/>
+    <axis xyz="0 0 1"/>
+    <origin xyz="-0.039 0.045 0.023" rpy="0 0 0"/>
     <limit effort="1" velocity="1" upper="3.1415" lower="-3.1415"/>
   </joint>
@@ -197,8 +195,6 @@
     <parent link="right_leg_upper_hip_link"/>
     <child link="right_leg_lower_hip_link"/>
-    <axis>
-      <xyz>0 1 0</xyz>
-    </axis>
-    <origin xyz="0.040 -0.045 -0.01" rpy="0 0 0"/>
+    <axis xyz="0 1 0"/>
+    <origin xyz="-0 0.053 -0.036" rpy="0 0 0"/>
     <limit effort="1" velocity="1" upper="3.1415" lower="-3.1415"/>
   </joint>
@@ -206,8 +202,6 @@
     <parent link="right_leg_lower_hip_link"/>
     <child link="right_leg_thigh_link"/>
-    <axis>
-      <xyz>-1 0 0</xyz>
-    </axis>
-    <origin xyz="0.040 -0.045 -0.01" rpy="0 0 0"/>
+    <axis xyz="1 0 0"/>
+    <origin xyz="0.015 -0.053 0" rpy="0 0 0"/>
     <limit effort="1" velocity="1" upper="3.1415" lower="-3.1415"/>
   </joint>
@@ -215,8 +209,6 @@
     <parent link="right_leg_thigh_link"/>
     <child link="right_leg_knee_link"/>
-    <axis>
-      <xyz>1 0 0</xyz>
-    </axis>
-    <origin xyz="0.015 -0.04 -0.09" rpy="0 0 0"/>
+    <axis xyz="1 0 0"/>
+    <origin xyz="0.006 -0.006 -0.077" rpy="0 0 0"/>
     <limit effort="1" velocity="1" upper="3.1415" lower="-3.1415"/>
   </joint>
@@ -224,8 +216,6 @@
     <parent link="right_leg_knee_link"/>
     <child link="right_leg_shin_link"/>
-    <axis>
-      <xyz>1 0 0</xyz>
-    </axis>
-    <origin xyz="0.015 -0.04 -0.09" rpy="0 0 0"/>
+    <axis xyz="1 0 0"/>
+    <origin xyz="-0.004 -0.002 -0.015" rpy="0 0 0"/>
     <limit effort="1" velocity="1" upper="3.1415" lower="-3.1415"/>
   </joint>
@@ -233,8 +223,6 @@
     <parent link="right_leg_shin_link"/>
     <child link="right_leg_ankle_link"/>
-    <axis>
-      <xyz>1 0 0</xyz>
-    </axis>
-    <origin xyz="0.015 -0.045 -0.16" rpy="0 0 0"/>
+    <axis xyz="1 0 0"/>
+    <origin xyz="0.004 0.008 -0.058" rpy="0 0 0"/>
     <limit effort="1" velocity="1" upper="3.1415" lower="-3.1415"/>
   </joint>
@@ -242,8 +230,6 @@
     <parent link="right_leg_ankle_link"/>
     <child link="right_leg_foot_link"/>
-    <axis>
-      <xyz>0 -1 0</xyz>
-    </axis>
-    <origin xyz="0.04 -0.045 -0.16" rpy="0 0 0"/>
+    <axis xyz="0 1 0"/>
+    <origin xyz="-0.021 0.053 0" rpy="0 0 0"/>
     <limit effort="1" velocity="1" upper="3.1415" lower="-3.1415"/>
   </joint>

File: hros1_description/urdf/hros1_robot.urdf (robot description, URDF)
Before this commit: robot hros1, 20 links, 19 joints
Links:
- added link right_arm_elbow_link, mass 0.016; visual mesh filename=package://hros1_description/meshes/right_arm_elbow_link.stl
- added link right_arm_forearm_servo_link, mass 0.055; visual mesh filename=package://hros1_description/meshes/right_arm_forearm_servo.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
- added link right_arm_shoulder_link, mass 0.011; visual mesh filename=package://hros1_description/meshes/right_arm_shoulder.stl
- added link right_arm_upper_servo_link, mass 0.055; visual mesh filename=package://hros1_description/meshes/right_arm_upper_servo.stl
- added link right_leg_ankle_link, mass 0.110; visual mesh filename=package://hros1_description/meshes/right_leg_ankle_joint.stl
- added link right_leg_foot_link, mass 0.067; collision box size=0.065 .1 0.01; visual mesh filename=package://hros1_description/meshes/right_leg_foot.stl
- added link right_leg_knee_link, mass 0.055; visual mesh filename=package://hros1_description/meshes/right_leg_knee.stl
- added link right_leg_lower_hip_link, mass 0.110; visual mesh filename=package://hros1_description/meshes/right_leg_hip_joint.stl
- added link right_leg_shin_link, mass 0.021; visual mesh filename=package://hros1_description/meshes/right_leg_shin.stl
- added link right_leg_thigh_link, mass 0.028; visual mesh filename=package://hros1_description/meshes/right_leg_thigh.stl
- added link right_leg_upper_hip_link, mass 0.017; visual mesh filename=package://hros1_description/meshes/right_leg_yaw_link.stl
- link left_arm_elbow_link: geometry visual mesh filename=package://hros1_description/meshes/left_arm_elbow_link.stl
- link left_arm_forearm_servo_link: geometry visual mesh filename=package://hros1_description/meshes/left_arm_forearm_servo.s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
- link left_arm_shoulder_link: geometry visual mesh filename=package://hros1_description/meshes/left_arm_shoulder.stl
- link left_arm_upper_servo_link: geometry visual mesh filename=package://hros1_description/meshes/left_arm_upper_servo.stl
- link left_leg_ankle_link: geometry visual mesh filename=package://hros1_description/meshes/left_leg_ankle_joint.stl
- link left_leg_foot_link: geometry collision box size=0.065 .1 0.01; visual mesh filename=package://hros1_description/meshes/left_leg_foot.stl
- link left_leg_knee_link: geometry visual mesh filename=package://hros1_description/meshes/left_leg_knee.stl
- link left_leg_lower_hip_link: geometry visual mesh filename=package://hros1_description/meshes/left_leg_hip_joint.stl
- link left_leg_shin_link: geometry visual mesh filename=package://hros1_description/meshes/left_leg_shin.stl
- link left_leg_thigh_link: geometry visual mesh filename=package://hros1_description/meshes/left_leg_thigh.stl
- link left_leg_upper_hip_link: geometry visual mesh filename=package://hros1_description/meshes/left_leg_yaw_link.stl
- link neck_base_link: geometry visual mesh filename=package://hros1_description/meshes/neck_base.stl
- link neck_base_platform_link: geometry collision cylinder length=0.0025 radius=0.02; visual mesh filename=package://hros1_description/meshes/neck_base_platform.stl
- link neck_head_link: geometry collision box size=0.02 0.02 0.02; visual mesh filename=package://hros1_description/meshes/neck_head_servo.stl
- link neck_link_1_link: geometry visual mesh filename=package://hros1_description/meshes/neck_link_1.stl
- link neck_link_2_link: geometry visual mesh filename=package://hros1_description/meshes/neck_link_2.stl
Joints:
- added joint right_ankle_pitch_powered_joint: type revolute, parent right_leg_shin_link, child right_leg_ankle_link, origin xyz=0.004 0.008 -0.058 rpy=0 0 0, axis 1 0 0, limit lower=-3.1415 upper=3.1415 effort=1 velocity=1
- added joint right_ankle_roll_powered_joint: type revolute, parent right_leg_ankle_link, child right_leg_foot_link, origin xyz=-0.021 0.053 0 rpy=0 0 0, axis 0 1 0, limit lower=-3.1415 upper=3.1415 effort=1 velocity=1
- added joint right_elbow_powered_joint: type revolute, parent right_arm_elbow_link, child right_arm_forearm_servo_link, origin xyz=0.005 0.0 -0.03 rpy=0 0 0, axis -0.8 0.0 -0.2, limit lower=-3.1415 upper=3.1415 effort=1 velocity=1
- added joint right_hip_pitch_powered_joint: type revolute, parent right_leg_lower_hip_link, child right_leg_thigh_link, origin xyz=0.015 -0.053 0 rpy=0 0 0, axis 1 0 0, limit lower=-3.1415 upper=3.1415 effort=1 velocity=1
- added joint right_hip_roll_powered_joint: type revolute, parent right_leg_upper_hip_link, child right_leg_lower_hip_link, origin xyz=-0 0.053 -0.036 rpy=0 0 0, axis 0 1 0, limit lower=-3.1415 upper=3.1415 effort=1 velocity=1
- added joint right_hip_yaw_powered_joint: type revolute, parent body_structure_link, child right_leg_upper_hip_link, origin xyz=-0.039 0.045 0.023 rpy=0 0 0, axis 0 0 1, limit lower=-3.1415 upper=3.1415 effort=1 velocity=1
- added joint right_knee-shin_fixed_joint: type fixed, parent right_leg_knee_link, child right_leg_shin_link, origin xyz=-0.004 -0.002 -0.015 rpy=0 0 0, axis 1 0 0, limit lower=-3.1415 upper=3.1415 effort=1 velocity=1
- added joint right_knee_pitch_powered_joint: type revolute, parent right_leg_thigh_link, child right_leg_knee_link, origin xyz=0.006 -0.006 -0.077 rpy=0 0 0, axis 1 0 0, limit lower=-3.1415 upper=3.1415 effort=1 velocity=1
- added joint right_shoulder-elbow_fixed_joint: type fixed, parent right_arm_upper_servo_link, child right_arm_elbow_link, origin xyz=-0.002 -0.033 -0.037 rpy=0 0 0, axis 0 -1 0
- added joint right_shoulder_pitch_powered_joint: type revolute, parent body_structure_link, child right_arm_shoulder_link, origin xyz=-0.051 0.052 0.133 rpy=0 0 0, axis -1 0 0, limit lower=-3.1415 upper=3.1415 effort=1 velocity=1
- added joint right_shoulder_roll_powered_joint: type revolute, parent right_arm_shoulder_link, child right_arm_upper_servo_link, origin xyz=-0.03 0.02 -0.015 rpy=0 0 0, axis 0 -1 0, limit lower=-3.1415 upper=3.1415 effort=1 velocity=1

File: hros1_description/urdf/hros1_robot.urdf.xacro (robot description, xacro)
@@ -6,8 +6,6 @@
     <xacro:include filename="$(find hros1_description)/urdf/hros1_left_arm.xacro"/>
     <xacro:include filename="$(find hros1_description)/urdf/hros1_left_leg.xacro"/>
-<!--
     <xacro:include filename="$(find hros1_description)/urdf/hros1_right_arm.xacro"/>
     <xacro:include filename="$(find hros1_description)/urdf/hros1_right_leg.xacro"/>
-  -->
     <xacro:body_links />
     <xacro:body_joints />
@@ -18,10 +16,8 @@
     <xacro:left_leg_links />
     <xacro:left_leg_joints />
-    <!--
     <xacro:right_arm_links />
     <xacro:right_arm_joints />
     <xacro:right_leg_links />
     <xacro:right_leg_joints />
-    -->
     <link name="world"/>
     <joint name="fixed_joint" type="fixed">
