Commit message: Model is now working with correct meshes and alignment of parts

File: hros1_description/urdf/hros1_right_arm.xacro (robot description, xacro)
@@ -126,5 +126,5 @@
     <parent link="right_arm_elbow_link"/>
     <child link="right_arm_forearm_servo_link"/>
-    <axis xyz="-0.8 0.0 -0.2"/>
+    <axis xyz="-0.8 0.0 0.2"/>
     <origin xyz="0.005 0.0 -0.03" rpy="0 0 0"/>
     <limit effort="1" velocity="1" upper="3.1415" lower="-3.1415"/>

File: hros1_description/urdf/hros1_robot.urdf (robot description, URDF)
Before this commit: robot hros1, 31 links, 30 joints
Joints:
- joint right_elbow_powered_joint: axis -0.8 0.0 -0.2 -> -0.8 0.0 0.2
