Commit message: Changed inertia tags

File: hros1_description/urdf/hros1_body.xacro (robot description, xacro)
@@ -31,15 +31,15 @@
         </geometry>
       </collision>
-      <inertial>
+      <inertial
         <pose>0 -0.065 0.082 0 -0 0</pose>
         <mass>0.273</mass>
-        <inertia>
-          <ixx>0.00074</ixx>
-          <ixy>-0.0000022</ixy>
-          <ixz>0.000000010</ixz>
-          <iyy>0.00088</iyy>
-          <iyz>0.000012</iyz>
-          <izz>0.00047</izz>
-          </inertia>
+        <inertia
+          ixx="0.00074"
+          ixy="-0.0000022"
+          ixz="0.000000010"
+          iyy="0.00088"
+          iyz="0.000012"
+          izz="0.00047"
+          />
       </inertial>
     </link>
@@ -66,15 +66,15 @@
         </material>
       </visual>
-      <inertial>
+      <inertial
         <pose>0 -0.055 0.086 0 -0 0</pose>
         <mass>0.221</mass>
-        <inertia>
-          <ixx>0.000056</ixx>
-          <ixy>0.000000068</ixy>
-          <ixz>0.00000015</ixz>
-          <iyy>0.00078</iyy>
-          <iyz>-0.00010</iyz>
-          <izz>0.00031</izz>
-          </inertia>
+        <inertia
+          ixx="0.000056"
+          ixy="0.000000068"
+          ixz="0.00000015"
+          iyy="0.00078"
+          iyz="-0.00010"
+          izz="0.00031"
+          />
       </inertial>
     </link>
@@ -104,12 +104,12 @@
         <pose>0 -0.078 0.036 0 -0 0</pose>
         <mass>0.25</mass>
-        <inertia>
-          <ixx>0.000037</ixx>
-          <ixy>-0.000000049</ixy>
-          <ixz>0.0</ixz>
-          <iyy>0.00026</iyy>
-          <iyz>0.0</iyz>
-          <izz>0.00027</izz>
-          </inertia>
+        <inertia
+          ixx="0.000037"
+          ixy="-0.000000049"
+          ixz="0.0</ixz>
+          iyy="0.00026"
+          iyz="0.0"
+          izz="0.00027"
+          />
       </inertial>
     </link>

Commit message: Changed visual and inertial elements of body file

File: hros1_description/urdf/hros1_body.xacro (robot description, xacro)
@@ -11,8 +11,5 @@
         <pose>0 0 0 0 -0 0</pose>
         <geometry>
-          <mesh>
-            <uri>model://HR-OS1/meshes/HROS1_Simple - Body_Structure.stl</uri>
-            <scale>1 1 1</scale>
-          </mesh>
+          <mesh filename="model://HR-OS1/meshes/HROS1_Simple - Body_Structure.stl"/>
         </geometry>
         <material>
@@ -31,7 +28,7 @@
         </geometry>
       </collision>
-      <inertial
-        <pose>0 -0.065 0.082 0 -0 0</pose>
-        <mass>0.273</mass>
+      <inertial>
+        <origin xyz="0 -0.065 0.082" rpy=" 0 -0 0"/>
+        <mass value="0.273"/>
         <inertia
           ixx="0.00074"
@@ -66,7 +63,7 @@
         </material>
       </visual>
-      <inertial
-        <pose>0 -0.055 0.086 0 -0 0</pose>
-        <mass>0.221</mass>
+      <inertial>
+        <origin xyz="0 -0.055 0.086" rpy=" 0 -0 0"/>
+        <mass value="0.221"/>
         <inertia
           ixx="0.000056"
@@ -102,10 +99,10 @@
       </visual>
       <inertial>
-        <pose>0 -0.078 0.036 0 -0 0</pose>
-        <mass>0.25</mass>
+        <origin xyz="0 -0.078 0.036" rpy=" 0 -0 0"/>
+        <mass value="0.25"/>
         <inertia
           ixx="0.000037"
           ixy="-0.000000049"
-          ixz="0.0</ixz>
+          ixz="0.0"
           iyy="0.00026"
           iyz="0.0"

File: hros1_description/urdf/hros1_neck.xacro (robot description, xacro)
@@ -1,4 +1,5 @@
 <?xml version="1.0"?>
 <robot xmlns:xacro="http://ros.org/wiki/xacro">
+test
 <xacro:macro name="neck_links">
     <!--  ATTACHED TO TOP OF BODY -->

File: hros1_description/urdf/hros1_robot.urdf.xacro (robot description, xacro)
@@ -10,4 +10,5 @@
     <xacro:body_links />
     <xacro:body_joints />
+    <!--
     <xacro:neck_links />
     <xacro:neck_joints />
@@ -20,3 +21,4 @@
     <xacro:right_leg_links />
     <xacro:right_leg_joints />
+    -->
 </robot>

Commit message: Changed visual filename tags of body file

File: hros1_description/urdf/hros1_body.xacro (robot description, xacro)
@@ -51,8 +51,5 @@
         <pose>0 0 0 0 -0 0</pose>
         <geometry>
-          <mesh>
-            <uri>model://HR-OS1/meshes/HROS1_Simple - Body_Servos.stl</uri>
-            <scale>1 1 1</scale>
-          </mesh>
+          <mesh filename="model://HR-OS1/meshes/HROS1_Simple - Body_Servos.stl"/>
         </geometry>
         <material>
@@ -86,8 +83,5 @@
         <pose>0 0 0 0 -0 0</pose>
         <geometry>
-          <mesh>
-            <uri>model://HR-OS1/meshes/HROS1_Simple - Body_Battery.stl</uri>
-            <scale>1 1 1</scale>
-          </mesh>
+          <mesh filename="model://HR-OS1/meshes/HROS1_Simple - Body_Battery.stl"/>
         </geometry>
         <material>

Commit message: Added size tag to collision element in body file

File: hros1_description/urdf/hros1_body.xacro (robot description, xacro)
@@ -25,7 +25,5 @@
         <pose> 0 -0.055 0.08 0 0 0 </pose>
         <geometry>
-          <box>
-            <size>0.08 0.07 0.12</size>
-          </box>
+          <box size="0.08 0.07 0.12"/>
         </geometry>
       </collision>

Commit message: Changed body filexacro-urdf tags; now working

File: hros1_description/urdf/hros1_body.xacro (robot description, xacro)
@@ -11,5 +11,5 @@
         <pose>0 0 0 0 -0 0</pose>
         <geometry>
-          <mesh filename="model://HR-OS1/meshes/HROS1_Simple - Body_Structure.stl"/>
+          <mesh filename="package://hros1_description/meshes/HROS1_Simple - Body_Structure.stl"/>
         </geometry>
         <!--
@@ -25,7 +25,5 @@
         <pose> 0 -0.055 0.08 0 0 0 </pose>
         <geometry>
-          <box>
-            <size>0.08 0.07 0.12</size>
-          </box>
+          <box size="0.08 0.07 0.12"/>
         </geometry>
       </collision>
@@ -53,5 +51,5 @@
         <pose>0 0 0 0 -0 0</pose>
         <geometry>
-          <mesh filename="model://HR-OS1/meshes/HROS1_Simple - Body_Servos.stl"/>
+          <mesh filename="package://hros1_description/meshes/HROS1_Simple - Body_Servos.stl"/>
         </geometry>
         <!--
@@ -87,5 +85,5 @@
         <pose>0 0 0 0 -0 0</pose>
         <geometry>
-          <mesh filename="model://HR-OS1/meshes/HROS1_Simple - Body_Battery.stl"/>
+          <mesh filename="package://hros1_description/meshes/HROS1_Simple - Body_Battery.stl"/>
         </geometry>
         <!--
@@ -113,7 +111,7 @@
 </xacro:macro>
 <xacro:macro name="body_joints">
-<joint name="body-servos_fixture_joint" type="revolute">
-    <parent>HR-OS1::body_structure_link</parent>
-    <child>HR-OS1::body_servos_link</child>
+<joint name="body-servos_fixture_joint" type="fixed">
+    <parent link="HR-OS1::body_structure_link"/>
+    <child link="HR-OS1::body_servos_link"/>
     <axis>
       <xyz>0 0 1</xyz>
@@ -124,7 +122,7 @@
     </axis>
   </joint>
-  <joint name="body-battery_fixture_joint" type="revolute">
-    <parent>HR-OS1::body_structure_link</parent>
-    <child>HR-OS1::body_battery_link</child>
+  <joint name="body-battery_fixture_joint" type="fixed">
+    <parent link="HR-OS1::body_structure_link"/>
+    <child link="HR-OS1::body_battery_link"/>
     <axis>
       <xyz>0 1 0</xyz>

Commit message: Changed pose tags in body file

File: hros1_description/urdf/hros1_body.xacro (robot description, xacro)
@@ -9,5 +9,5 @@
       <kinematic>0</kinematic>
       <visual name='body_structure_visual'>
-        <pose>0 0 0 0 -0 0</pose>
+        <origin xyz="0 0 0"  rpy="0 -0 0"/>
         <geometry>
           <mesh filename="package://hros1_description/meshes/HROS1_Simple - Body_Structure.stl"/>
@@ -23,5 +23,5 @@
       </visual>
       <collision name="collision">
-        <pose> 0 -0.055 0.08 0 0 0 </pose>
+        <origin xyz="0 -0.055 0.08" rpy="0 0 0"/>
         <geometry>
           <box size="0.08 0.07 0.12"/>
@@ -44,5 +44,5 @@
 <!--  JOINTS CONNECTED HERE  -->
     <link name='HR-OS1::body_servos_link'>
-      <pose>0 0 0 0 -0 0</pose>
+      <origin xyz="0 0 0" rpy="0 -0 0"/>
       <gravity>1</gravity>
       <self_collide>0</self_collide>
@@ -78,10 +78,10 @@
 <!--  ADDED FOR WEIGHT  -->
     <link name='HR-OS1::body_battery_link'>
-      <pose>0 0 0 0 -0 0</pose>
+      <origin xyz="0 0 0" rpy"0 -0 0"/>
       <gravity>0</gravity>
       <self_collide>0</self_collide>
       <kinematic>0</kinematic>
       <visual name='body_battery_visual'>
-        <pose>0 0 0 0 -0 0</pose>
+        <origin xyz="0 0 0" rpy="0 -0 0"/>
         <geometry>
           <mesh filename="package://hros1_description/meshes/HROS1_Simple - Body_Battery.stl"/>

Commit message: Made changes to neck file

File: hros1_description/urdf/hros1_body.xacro (robot description, xacro)
@@ -78,5 +78,5 @@
 <!--  ADDED FOR WEIGHT  -->
     <link name='HR-OS1::body_battery_link'>
-      <origin xyz="0 0 0" rpy"0 -0 0"/>
+      <origin xyz="0 0 0" rpy="0 -0 0"/>
       <gravity>0</gravity>
       <self_collide>0</self_collide>

File: hros1_description/urdf/hros1_neck.xacro (robot description, xacro)
@@ -10,26 +10,20 @@
       <kinematic>0</kinematic>
       <visual name='neck_link_1_visual'>
-        <origin xyz="0 0 0 0 -0 0"/>
+        <origin xyz="0 0 0" rpy="0 -0 0"/>
         <geometry>
           <mesh filename="package://hros1_description/meshes/HROS1_Simple - Neck_Link_1.stl"/>
         </geometry>
-        <material>
-          <script>
-            <uri>file://media/materials/scripts/gazebo.material"
-            <name>Gazebo/Grey</name>
-          </script>
-        </material>
       </visual>
       <inertial>
-        <origin xyz="0 -0.101 0.208 0 -0 0"/>
-        <mass>0.005</mass>
-        <inertia>
-          <ixx>0.0000012</ixx>
-          <ixy>0.0</ixy>
-          <ixz>0.0</ixz>
-          <iyy>0.0000032</iyy>
-          <iyz>0.0</iyz>
-          <izz>0.000002</izz>
-          </inertia>
+        <origin xyz="0 -0.101 0.208" rpy="0 -0 0"/>
+        <mass value="0.005"/>
+        <inertia
+          ixx="0.0000012"
+          ixy="0.0"
+          ixz="0.0"
+          iyy="0.0000032"
+          iyz="0.0"
+          izz="0.000002"
+          />
       </inertial>
     </link>
@@ -37,6 +31,7 @@
 <xacro:macro name="neck_joints">
   <joint name="neck_yaw_powered_joint" type="revolute">
-    <parent>HR-OS1::body_structure_link</parent>
-    <child>HR-OS1::neck_base_link</child>
+    <parent link="HR-OS1::body_structure_link"/>
+    <child link="HR-OS1::neck_base_link"/>
+    <limit effort="1" velocity="1" lower="-3.1415" upper="3.1415"/>
     <axis>
       <xyz>0 0 1</xyz>
@@ -45,6 +40,7 @@
   </joint>
   <joint name="neck_base_platform_free_joint" type="revolute">
-    <parent>HR-OS1::neck_base_link</parent>
-    <child>HR-OS1::neck_base_platform_link</child>
+    <parent link="HR-OS1::neck_base_link"/>
+    <child link="HR-OS1::neck_base_platform_link"/>
+    <limit effort="1" velocity="1" upper="3.1415" lower="-3.1415"/>
     <axis>
       <xyz>1 0 0</xyz>
@@ -53,6 +49,7 @@
   </joint>
   <joint name="neck_pitch_1_free_joint" type="revolute">
-    <parent>HR-OS1::neck_base_link</parent>
-    <child>HR-OS1::neck_link_1_link</child>
+    <parent link="HR-OS1::neck_base_link"/>
+    <child link="HR-OS1::neck_link_1_link"/>
+    <limit effort="1" velocity="1" upper="3.1415" lower="-3.1415"/>
     <axis>
       <xyz>1 0 0</xyz>
@@ -61,6 +58,7 @@
   </joint>
   <joint name="neck_pitch_2_free_joint" type="revolute">
-    <parent>HR-OS1::neck_link_1_link</parent>
-    <child>HR-OS1::neck_link_2_link</child>
+    <parent link="HR-OS1::neck_link_1_link"/>
+    <child link="HR-OS1::neck_link_2_link"/>
+    <limit effort="1" velocity="1" upper="3.1415" lower="-3.1415"/>
     <axis>
       <xyz>1 0 0</xyz>
@@ -69,6 +67,7 @@
   </joint>
   <joint name="neck_pitch_main_powered_joint" type="revolute">
-    <parent>HR-OS1::neck_link_2_link</parent>
-    <child>HR-OS1::neck_head_link</child>
+    <parent link="HR-OS1::neck_link_2_link"/>
+    <child link="HR-OS1::neck_head_link"/>
+    <limit effort="1" velocity="1" upper="3.1415" lower="-3.1415"/>
     <axis>
       <xyz>-1 0 0</xyz>

File: hros1_description/urdf/hros1_robot.urdf.xacro (robot description, xacro)
@@ -10,7 +10,7 @@
     <xacro:body_links />
     <xacro:body_joints />
-    <!--
     <xacro:neck_links />
     <xacro:neck_joints />
+    <!--
     <xacro:left_arm_links />
     <xacro:left_arm_joints />

Commit message: Changed box collision tags

File: hros1_description/urdf/hros1_body.xacro (robot description, xacro)
@@ -53,12 +53,4 @@
           <mesh filename="package://hros1_description/meshes/HROS1_Simple - Body_Servos.stl"/>
         </geometry>
-        <!--
-        <material>
-          <script>
-            <uri>file://media/materials/scripts/gazebo.material</uri>
-            <name>Gazebo/Grey</name>
-          </script>
-        </material>
-        -->
       </visual>
       <inertial>
@@ -87,12 +79,4 @@
           <mesh filename="package://hros1_description/meshes/HROS1_Simple - Body_Battery.stl"/>
         </geometry>
-        <!--
-        <material>
-          <script>
-            <uri>file://media/materials/scripts/gazebo.material</uri>
-            <name>Gazebo/Grey</name>
-          </script>
-        </material>
-        -->
       </visual>
       <inertial>

File: hros1_description/urdf/hros1_neck.xacro (robot description, xacro)
@@ -17,7 +17,5 @@
         <origin xyz=" 0.0 -0.05 0.22" rpy="0 0 0 "/>
         <geometry>
-          <box>
-            <size>0.02 0.02 0.02</size>
-          </box>
+          <box size="0.02 0.02 0.02"/>
         </geometry>
       </collision>
