Commit message: Added arm/leg imports to body xacro; removed HR-OS1:: from link names

File: hros1_description/urdf/hros1_body.xacro (robot description, xacro)
@@ -4,5 +4,5 @@
 <!--  MAIN BODY  -->
 <!--  MAIN LINK  -->
-    <link name='HR-OS1::body_structure_link'>
+    <link name='body_structure_link'>
       <gravity>1</gravity>
       <self_collide>0</self_collide>
@@ -43,5 +43,5 @@
 <!--  SERVOS ON BODY  -->
 <!--  JOINTS CONNECTED HERE  -->
-    <link name='HR-OS1::body_servos_link'>
+    <link name='body_servos_link'>
       <origin xyz="0 0 0" rpy="0 -0 0"/>
       <gravity>1</gravity>
@@ -69,5 +69,5 @@
 <!--  MAIN BATTERY  -->
 <!--  ADDED FOR WEIGHT  -->
-    <link name='HR-OS1::body_battery_link'>
+    <link name='body_battery_link'>
       <origin xyz="0 0 0" rpy="0 -0 0"/>
       <gravity>0</gravity>
@@ -96,6 +96,6 @@
 <xacro:macro name="body_joints">
 <joint name="body-servos_fixture_joint" type="fixed">
-    <parent link="HR-OS1::body_structure_link"/>
-    <child link="HR-OS1::body_servos_link"/>
+    <parent link="body_structure_link"/>
+    <child link="body_servos_link"/>
     <axis>
       <xyz>0 0 1</xyz>
@@ -107,6 +107,6 @@
   </joint>
   <joint name="body-battery_fixture_joint" type="fixed">
-    <parent link="HR-OS1::body_structure_link"/>
-    <child link="HR-OS1::body_battery_link"/>
+    <parent link="body_structure_link"/>
+    <child link="body_battery_link"/>
     <axis>
       <xyz>0 1 0</xyz>

File: hros1_description/urdf/hros1_left_arm.xacro (robot description, xacro)
@@ -3,5 +3,5 @@
 <xacro:macro name="left_arm_links">
 <!--  LEFT ARM SHOULDER  -->
-    <link name='HR-OS1::left_arm_shoulder_link'>
+    <link name='left_arm_shoulder_link'>
       <origin xyz="0 0 0" rpy="0 -0 0"/>
       <gravity>1</gravity>
@@ -28,5 +28,5 @@
     </link>
 <!--  LEFT ARM UPPER SERVO  -->
-    <link name='HR-OS1::left_arm_upper_servo_link'>
+    <link name='left_arm_upper_servo_link'>
       <origin xyz="0 0 0 0 -0 0"/>
       <gravity>1</gravity>
@@ -53,5 +53,5 @@
     </link>
 <!--  LEFT ARM Elbow  -->
-    <link name='HR-OS1::left_arm_elbow_link'>
+    <link name='left_arm_elbow_link'>
       <origin xyz="0 0 0" rpy="0 -0 0"/>
       <gravity>1</gravity>
@@ -78,5 +78,5 @@
     </link>
 <!--  LEFT ARM FOREARM SERVO  -->
-    <link name='HR-OS1::left_arm_forearm_servo_link'>
+    <link name='left_arm_forearm_servo_link'>
       <origin xyz="0 0 0" rpy="0 -0 0"/>
       <gravity>1</gravity>
@@ -105,6 +105,6 @@
 <xacro:macro name="left_arm_joints">
   <joint name="left_shoulder_pitch_powered_joint" type="revolute">
-    <parent link="HR-OS1::body_structure_link"/>
-    <child link="HR-OS1::left_arm_shoulder_link"/>
+    <parent link="body_structure_link"/>
+    <child link="left_arm_shoulder_link"/>
     <axis>
       <xyz>-1 0 0</xyz>
@@ -114,6 +114,6 @@
   </joint>
   <joint name="left_shoulder_roll_powered_joint" type="revolute">
-    <parent link="HR-OS1::left_arm_shoulder_link"/>
-    <child link="HR-OS1::left_arm_upper_servo_link"/>
+    <parent link="left_arm_shoulder_link"/>
+    <child link="left_arm_upper_servo_link"/>
     <axis>
       <xyz>0 -1 0</xyz>
@@ -123,6 +123,6 @@
   </joint>
   <joint name="left_shoulder-elbow_fixed_joint" type="revolute">
-    <parent link="HR-OS1::left_arm_upper_servo_link"/>
-    <child link="HR-OS1::left_arm_elbow_link"/>
+    <parent link="left_arm_upper_servo_link"/>
+    <child link="left_arm_elbow_link"/>
     <axis>
       <xyz>0 1 0</xyz>
@@ -134,6 +134,6 @@
   </joint>
   <joint name="left_elbow_powered_joint" type="revolute">
-    <parent link="HR-OS1::left_arm_elbow_link"/>
-    <child link="HR-OS1::left_arm_forearm_servo_link"/>
+    <parent link="left_arm_elbow_link"/>
+    <child link="left_arm_forearm_servo_link"/>
     <axis>
       <xyz>1 0 -0.25</xyz>

File: hros1_description/urdf/hros1_left_leg.xacro (robot description, xacro)
@@ -3,5 +3,5 @@
 <xacro:macro name="left_leg_links">
 <!-- LEFT Upper HIP  -->
-    <link name='HR-OS1::left_leg_upper_hip_link'>
+    <link name='left_leg_upper_hip_link'>
       <origin xyz="0 0 0" rpy="0 -0 0"/>
       <gravity>1</gravity>
@@ -28,5 +28,5 @@
     </link>
 <!-- LEFT LOWER HIP  -->
-    <link name='HR-OS1::left_leg_lower_hip_link'>
+    <link name='left_leg_lower_hip_link'>
       <origin xyz="0 0 0 0 -0 0"/>
       <gravity>1</gravity>
@@ -53,5 +53,5 @@
     </link>
 <!-- LEFT THIGH  -->
-    <link name='HR-OS1::left_leg_thigh_link'>
+    <link name='left_leg_thigh_link'>
       <origin xyz="0 0 0 0 -0 0"/>
       <gravity>1</gravity>
@@ -78,5 +78,5 @@
     </link>
 <!-- LEFT KNEE  -->
-    <link name='HR-OS1::left_leg_knee_link'>
+    <link name='left_leg_knee_link'>
       <origin xyz="0 0 0" rpy="0 -0 0"/>
       <gravity>1</gravity>
@@ -103,5 +103,5 @@
     </link>
 <!-- LEFT SHIN  -->
-    <link name='HR-OS1::left_leg_shin_link'>
+    <link name='left_leg_shin_link'>
       <origin xyz="0 0 0" rpy="0 -0 0"/>
       <gravity>1</gravity>
@@ -128,5 +128,5 @@
     </link>
 <!-- LEFT ANKLE  -->
-    <link name='HR-OS1::left_leg_ankle_link'>
+    <link name='left_leg_ankle_link'>
       <origin xyz="0 0 0" rpy="0 -0 0"/>
       <gravity>1</gravity>
@@ -153,5 +153,5 @@
     </link>
 <!-- LEFT FOOT  -->
-    <link name='HR-OS1::left_leg_foot_link'>
+    <link name='left_leg_foot_link'>
       <origin xyz="0 0 0" rpy="0 -0 0"/>
       <gravity>1</gravity>
@@ -167,7 +167,5 @@
         <origin xyz=" -0.05 -0.05 -0.195" rpy="0 0 0 "/>
         <geometry>
-          <box>
-            <size>0.065 .1 0.01</size>
-          </box>
+          <box size="0.065 .1 0.01"/>
         </geometry>
       </collision>
@@ -188,6 +186,6 @@
 <xacro:macro name="left_leg_joints">
   <joint name="left_hip_yaw_powered_joint" type="revolute">
-    <parent link="HR-OS1::body_structure_link"/>
-    <child link="HR-OS1::left_leg_upper_hip_link"/>
+    <parent link="body_structure_link"/>
+    <child link="left_leg_upper_hip_link"/>
     <axis>
       <xyz>0 0 -1</xyz>
@@ -197,6 +195,6 @@
   </joint>
   <joint name="left_hip_roll_powered_joint" type="revolute">
-    <parent link="HR-OS1::left_leg_upper_hip_link"/>
-    <child link="HR-OS1::left_leg_lower_hip_link"/>
+    <parent link="left_leg_upper_hip_link"/>
+    <child link="left_leg_lower_hip_link"/>
     <axis>
       <xyz>0 1 0</xyz>
@@ -206,6 +204,6 @@
   </joint>
   <joint name="left_hip_pitch_powered_joint" type="revolute">
-    <parent link="HR-OS1::left_leg_lower_hip_link"/>
-    <child link="HR-OS1::left_leg_thigh_link"/>
+    <parent link="left_leg_lower_hip_link"/>
+    <child link="left_leg_thigh_link"/>
     <axis>
       <xyz>1 0 0</xyz>
@@ -215,6 +213,6 @@
   </joint>
   <joint name="left_knee_pitch_powered_joint" type="revolute">
-    <parent link="HR-OS1::left_leg_thigh_link"/>
-    <child link="HR-OS1::left_leg_knee_link"/>
+    <parent link="left_leg_thigh_link"/>
+    <child link="left_leg_knee_link"/>
     <axis>
       <xyz>-1 0 0</xyz>
@@ -224,6 +222,6 @@
   </joint>
   <joint name="left_knee-shin_fixed_joint" type="revolute">
-    <parent link="HR-OS1::left_leg_knee_link"/>
-    <child link="HR-OS1::left_leg_shin_link"/>
+    <parent link="left_leg_knee_link"/>
+    <child link="left_leg_shin_link"/>
     <axis>
       <xyz>1 0 0</xyz>
@@ -237,6 +235,6 @@
   </joint>
   <joint name="left_ankle_pitch_powered_joint" type="revolute">
-    <parent link="HR-OS1::left_leg_shin_link"/>
-    <child link="HR-OS1::left_leg_ankle_link"/>
+    <parent link="left_leg_shin_link"/>
+    <child link="left_leg_ankle_link"/>
     <axis>
       <xyz>-1 0 0</xyz>
@@ -246,6 +244,6 @@
   </joint>
   <joint name="left_ankle_roll_powered_joint" type="revolute">
-    <parent link="HR-OS1::left_leg_ankle_link"/>
-    <child link="HR-OS1::left_leg_foot_link"/>
+    <parent link="left_leg_ankle_link"/>
+    <child link="left_leg_foot_link"/>
     <axis>
       <xyz>0 -1 0</xyz>

File: hros1_description/urdf/hros1_neck.xacro (robot description, xacro)
@@ -3,5 +3,5 @@
 <!--  NECK Head (Pitch Servo) -->
 <!--  ATTACHED TO BACK OF HEAD  -->
-    <link name='HR-OS1::neck_head_link'>
+    <link name='neck_head_link'>
       <origin xyz="0 0 0" rpy="0 -0 0"/>
       <gravity>1</gravity>
@@ -34,5 +34,5 @@
 <!--  NECK Base (YAW SERVO) -->
 <!--  ATTACHED TO BACK OF HEAD  -->
-    <link name='HR-OS1::neck_base_link'>
+    <link name='neck_base_link'>
       <origin xyz="0 0 0" rpy="0 -0 0"/>
       <gravity>1</gravity>
@@ -60,5 +60,5 @@
 <!--  Neck Head Platform  -->
 <!--  Supports to head; should be able to tilt  -->
-    <link name='HR-OS1::neck_base_platform_link'>
+    <link name='neck_base_platform_link'>
       <origin xyz="0 0 0" rpy="0 -0 0"/>
       <gravity>1</gravity>
@@ -92,5 +92,5 @@
 <!--  NECK Link 2  -->
 <!--  ATTACHED TO Head Servo  -->
-    <link name='HR-OS1::neck_link_2_link'>
+    <link name='neck_link_2_link'>
       <origin xyz="0 0 0" rpy="0 -0 0"/>
       <gravity>1</gravity>
@@ -118,5 +118,5 @@
 <xacro:macro name="neck_links">
     <!--  ATTACHED TO TOP OF BODY -->
-    <link name='HR-OS1::neck_link_1_link'>
+    <link name='neck_link_1_link'>
       <origin xyz="0 0 0" rpy="0 -0 0"/>
       <gravity>1</gravity>
@@ -145,6 +145,6 @@
 <xacro:macro name="neck_joints">
   <joint name="neck_yaw_powered_joint" type="revolute">
-    <parent link="HR-OS1::body_structure_link"/>
-    <child link="HR-OS1::neck_base_link"/>
+    <parent link="body_structure_link"/>
+    <child link="neck_base_link"/>
     <limit effort="1" velocity="1" lower="-3.1415" upper="3.1415"/>
     <axis>
@@ -154,6 +154,6 @@
   </joint>
   <joint name="neck_base_platform_free_joint" type="revolute">
-    <parent link="HR-OS1::neck_base_link"/>
-    <child link="HR-OS1::neck_base_platform_link"/>
+    <parent link="neck_base_link"/>
+    <child link="neck_base_platform_link"/>
     <limit effort="1" velocity="1" upper="3.1415" lower="-3.1415"/>
     <axis>
@@ -163,6 +163,6 @@
   </joint>
   <joint name="neck_pitch_1_free_joint" type="revolute">
-    <parent link="HR-OS1::neck_base_link"/>
-    <child link="HR-OS1::neck_link_1_link"/>
+    <parent link="neck_base_link"/>
+    <child link="neck_link_1_link"/>
     <limit effort="1" velocity="1" upper="3.1415" lower="-3.1415"/>
     <axis>
@@ -172,6 +172,6 @@
   </joint>
   <joint name="neck_pitch_2_free_joint" type="revolute">
-    <parent link="HR-OS1::neck_link_1_link"/>
-    <child link="HR-OS1::neck_link_2_link"/>
+    <parent link="neck_link_1_link"/>
+    <child link="neck_link_2_link"/>
     <limit effort="1" velocity="1" upper="3.1415" lower="-3.1415"/>
     <axis>
@@ -181,6 +181,6 @@
   </joint>
   <joint name="neck_pitch_main_powered_joint" type="revolute">
-    <parent link="HR-OS1::neck_link_2_link"/>
-    <child link="HR-OS1::neck_head_link"/>
+    <parent link="neck_link_2_link"/>
+    <child link="neck_head_link"/>
     <limit effort="1" velocity="1" upper="3.1415" lower="-3.1415"/>
     <axis>

File: hros1_description/urdf/hros1_right_arm.xacro (robot description, xacro)
@@ -2,5 +2,5 @@
 <robot xmlns:xacro="http://ros.org/wiki/xacro">
 <xacro:macro name="right_arm_links">
-	<link name='HR-OS1::right_arm_shoulder_link'>
+	<link name='right_arm_shoulder_link'>
       <origin xyz="0 0 0" rpy="0 -0 0"/>
       <gravity>1</gravity>
@@ -27,5 +27,5 @@
     </link>
 <!--  RIGHT UPPER SERVO  -->
-    <link name='HR-OS1::right_arm_upper_servo_link'>
+    <link name='right_arm_upper_servo_link'>
       <origin xyz="0 0 0" rpy="0 -0 0"/>
       <gravity>1</gravity>
@@ -52,5 +52,5 @@
     </link>
 <!--  RIGHT ELBOW  -->
-    <link name='HR-OS1::right_arm_elbow_link'>
+    <link name='right_arm_elbow_link'>
       <origin xyz="0 0 0" rpy="0 -0 0"/>
       <gravity>1</gravity>
@@ -77,5 +77,5 @@
     </link>
 <!--  RIGHT HAND SERVO  -->
-    <link name='HR-OS1::right_arm_forearm_servo_link'>
+    <link name='right_arm_forearm_servo_link'>
       <origin xyz="0 0 0" rpy="0 -0 0"/>
       <gravity>1</gravity>
@@ -104,6 +104,6 @@
 <xacro:macro name="right_arm_joints">
   <joint name="right_shoulder_pitch_powered_joint" type="revolute">
-    <parent link="HR-OS1::body_structure_link"/>
-    <child link="HR-OS1::right_arm_shoulder_link"/>
+    <parent link="body_structure_link"/>
+    <child link="right_arm_shoulder_link"/>
     <axis>
       <xyz>1 0 0</xyz>
@@ -113,6 +113,6 @@
   </joint>
   <joint name="right_shoulder_roll_powered_joint" type="revolute">
-    <parent link="HR-OS1::right_arm_shoulder_link"/>
-    <child link="HR-OS1::right_arm_upper_servo_link"/>
+    <parent link="right_arm_shoulder_link"/>
+    <child link="right_arm_upper_servo_link"/>
     <axis>
       <xyz>0 -1 0</xyz>
@@ -122,6 +122,6 @@
   </joint>
   <joint name="right_shoulder-elbow_fixed_joint" type="revolute">
-    <parent link="HR-OS1::right_arm_upper_servo_link"/>
-    <child link="HR-OS1::right_arm_elbow_link"/>
+    <parent link="right_arm_upper_servo_link"/>
+    <child link="right_arm_elbow_link"/>
     <axis>
       <xyz>0 1 0</xyz>
@@ -133,6 +133,6 @@
   </joint>
   <joint name="right_elbow_powered_joint" type="revolute">
-    <parent link="HR-OS1::right_arm_elbow_link"/>
-    <child link="HR-OS1::right_arm_forearm_servo_link"/>
+    <parent link="right_arm_elbow_link"/>
+    <child link="right_arm_forearm_servo_link"/>
     <axis>
       <xyz>-1 0 -0.25</xyz>

File: hros1_description/urdf/hros1_right_leg.xacro (robot description, xacro)
@@ -3,5 +3,5 @@
 <xacro:macro name="right_leg_links">
 	<!-- RIGHT Upper HIP  -->
-    <link name='HR-OS1::right_leg_upper_hip_link'>
+    <link name='right_leg_upper_hip_link'>
       <origin xyz="0 0 0" rpy="0 -0 0"/>
       <gravity>1</gravity>
@@ -28,5 +28,5 @@
     </link>
 <!-- RIGHT HIP  -->
-    <link name='HR-OS1::right_leg_lower_hip_link'>
+    <link name='right_leg_lower_hip_link'>
       <origin xyz="0 0 0" rpy="0 -0 0"/>
       <gravity>1</gravity>
@@ -53,5 +53,5 @@
     </link>
 <!-- RIGHT THIGH  -->
-    <link name='HR-OS1::right_leg_thigh_link'>
+    <link name='right_leg_thigh_link'>
       <origin xyz="0 0 0" rpy="0 -0 0"/>
       <gravity>1</gravity>
@@ -78,5 +78,5 @@
     </link>
 <!-- RIGHT KNEE  -->
-    <link name='HR-OS1::right_leg_knee_link'>
+    <link name='right_leg_knee_link'>
       <origin xyz="0 0 0" rpy="0 -0 0"/>
       <gravity>1</gravity>
@@ -103,5 +103,5 @@
     </link>
 <!-- RIGHT SHIN  -->
-    <link name='HR-OS1::right_leg_shin_link'>
+    <link name='right_leg_shin_link'>
       <origin xyz="0 0 0" rpy="0 -0 0"/>
       <gravity>1</gravity>
@@ -128,5 +128,5 @@
     </link>
 <!-- RIGHT ANKLE  -->
-    <link name='HR-OS1::right_leg_ankle_link'>
+    <link name='right_leg_ankle_link'>
       <origin xyz="0 0 0" rpy="0 -0 0"/>
       <gravity>1</gravity>
@@ -153,5 +153,5 @@
     </link>
 <!-- RIGHT FOOT  -->
-    <link name='HR-OS1::right_leg_foot_link'>
+    <link name='right_leg_foot_link'>
       <origin xyz="0 0 0" rpy="0 -0 0"/>
       <gravity>1</gravity>
@@ -188,6 +188,6 @@
 <xacro:macro name="right_leg_joints">
 <joint name="right_hip_yaw_powered_joint" type="revolute">
-    <parent link="HR-OS1::body_structure_link"/>
-    <child link="HR-OS1::right_leg_upper_hip_link"/>
+    <parent link="body_structure_link"/>
+    <child link="right_leg_upper_hip_link"/>
     <axis>
       <xyz>0 0 -1</xyz>
@@ -197,6 +197,6 @@
   </joint>
   <joint name="right_hip_roll_powered_joint" type="revolute">
-    <parent link="HR-OS1::right_leg_upper_hip_link"/>
-    <child link="HR-OS1::right_leg_lower_hip_link"/>
+    <parent link="right_leg_upper_hip_link"/>
+    <child link="right_leg_lower_hip_link"/>
     <axis>
       <xyz>0 1 0</xyz>
@@ -206,6 +206,6 @@
   </joint>
   <joint name="right_hip_pitch_powered_joint" type="revolute">
-    <parent link="HR-OS1::right_leg_lower_hip_link"/>
-    <child link="HR-OS1::right_leg_thigh_link"/>
+    <parent link="right_leg_lower_hip_link"/>
+    <child link="right_leg_thigh_link"/>
     <axis>
       <xyz>-1 0 0</xyz>
@@ -215,6 +215,6 @@
   </joint>
   <joint name="right_knee_pitch_powered_joint" type="revolute">
-    <parent link="HR-OS1::right_leg_thigh_link"/>
-    <child link="HR-OS1::right_leg_knee_link"/>
+    <parent link="right_leg_thigh_link"/>
+    <child link="right_leg_knee_link"/>
     <axis>
       <xyz>1 0 0</xyz>
@@ -224,6 +224,6 @@
   </joint>
   <joint name="right_knee-shin_fixed_joint" type="revolute">
-    <parent link="HR-OS1::right_leg_knee_link"/>
-    <child link="HR-OS1::right_leg_shin_link"/>
+    <parent link="right_leg_knee_link"/>
+    <child link="right_leg_shin_link"/>
     <axis>
       <xyz>1 0 0</xyz>
@@ -237,6 +237,6 @@
   </joint>
   <joint name="right_ankle_pitch_powered_joint" type="revolute">
-    <parent link="HR-OS1::right_leg_shin_link"/>
-    <child link="HR-OS1::right_leg_ankle_link"/>
+    <parent link="right_leg_shin_link"/>
+    <child link="right_leg_ankle_link"/>
     <axis>
       <xyz>1 0 0</xyz>
@@ -246,6 +246,6 @@
   </joint>
   <joint name="right_ankle_roll_powered_joint" type="revolute">
-    <parent link="HR-OS1::right_leg_ankle_link"/>
-    <child link="HR-OS1::right_leg_foot_link"/>
+    <parent link="right_leg_ankle_link"/>
+    <child link="right_leg_foot_link"/>
     <axis>
       <xyz>0 -1 0</xyz>

File: hros1_description/urdf/hros1_robot.urdf.xacro (robot description, xacro)
@@ -12,5 +12,4 @@
     <xacro:neck_links />
     <xacro:neck_joints />
-    <!--
     <xacro:left_arm_links />
     <xacro:left_arm_joints />
@@ -21,4 +20,3 @@
     <xacro:right_leg_links />
     <xacro:right_leg_joints />
-    -->
 </robot>

Commit message: Added fixed and continuous joint tags

File: hros1_description/urdf/hros1_body.xacro (robot description, xacro)
@@ -100,8 +100,4 @@
     <axis>
       <xyz>0 0 1</xyz>
-        <limit>
-          <lower>0</lower>
-          <upper>0</upper>
-        </limit>
     </axis>
   </joint>
@@ -111,8 +107,4 @@
     <axis>
       <xyz>0 1 0</xyz>
-        <limit>
-          <lower>0</lower>
-          <upper>0</upper>
-        </limit>
     </axis>
   </joint>

File: hros1_description/urdf/hros1_left_arm.xacro (robot description, xacro)
@@ -122,13 +122,8 @@
     <limit effort="1" velocity="1" upper="3.1415" lower="-3.1415"/>
   </joint>
-  <joint name="left_shoulder-elbow_fixed_joint" type="revolute">
+  <joint name="left_shoulder-elbow_fixed_joint" type="fixed">
     <parent link="left_arm_upper_servo_link"/>
     <child link="left_arm_elbow_link"/>
     <axis>
-      <xyz>0 1 0</xyz>
-      <limit>
-          <lower>0</lower>
-          <upper>0</upper>
-      </limit>
     </axis>
   </joint>

File: hros1_description/urdf/hros1_neck.xacro (robot description, xacro)
@@ -153,8 +153,8 @@
     <origin xyz="0 -0.045 0" rpy="0 0 0"/>
   </joint>
-  <joint name="neck_base_platform_free_joint" type="revolute">
+  <joint name="neck_base_platform_free_joint" type="continuous">
     <parent link="neck_base_link"/>
     <child link="neck_base_platform_link"/>
-    <limit effort="1" velocity="1" upper="3.1415" lower="-3.1415"/>
+    <limit effort="0" velocity="1" upper="3.1415" lower="-3.1415"/>
     <axis>
       <xyz>1 0 0</xyz>
@@ -162,8 +162,8 @@
     <origin xyz="0 -0.046 0.2" rpy="0 0 0"/>
   </joint>
-  <joint name="neck_pitch_1_free_joint" type="revolute">
+  <joint name="neck_pitch_1_free_joint" type="continuous">
     <parent link="neck_base_link"/>
     <child link="neck_link_1_link"/>
-    <limit effort="1" velocity="1" upper="3.1415" lower="-3.1415"/>
+    <limit effort="0" velocity="1" upper="3.1415" lower="-3.1415"/>
     <axis>
       <xyz>1 0 0</xyz>
@@ -171,8 +171,8 @@
     <origin xyz="0 -0.105 0.19" rpy="0 0 0"/>
   </joint>
-  <joint name="neck_pitch_2_free_joint" type="revolute">
+  <joint name="neck_pitch_2_free_joint" type="continuous">
     <parent link="neck_link_1_link"/>
     <child link="neck_link_2_link"/>
-    <limit effort="1" velocity="1" upper="3.1415" lower="-3.1415"/>
+    <limit effort="0" velocity="1" upper="3.1415" lower="-3.1415"/>
     <axis>
       <xyz>1 0 0</xyz>

File: hros1_description/urdf/hros1_right_arm.xacro (robot description, xacro)
@@ -121,13 +121,9 @@
     <limit effort="1" velocity="1" upper="3.1415" lower="-3.1415"/>
   </joint>
-  <joint name="right_shoulder-elbow_fixed_joint" type="revolute">
+  <joint name="right_shoulder-elbow_fixed_joint" type="fixed">
     <parent link="right_arm_upper_servo_link"/>
     <child link="right_arm_elbow_link"/>
     <axis>
       <xyz>0 1 0</xyz>
-      <limit>
-          <lower>0</lower>
-          <upper>0</upper>
-      </limit>
     </axis>
   </joint>

File: hros1_description/urdf/hros1_right_leg.xacro (robot description, xacro)
@@ -223,13 +223,9 @@
     <limit effort="1" velocity="1" upper="3.1415" lower="-3.1415"/>
   </joint>
-  <joint name="right_knee-shin_fixed_joint" type="revolute">
+  <joint name="right_knee-shin_fixed_joint" type="fixed">
     <parent link="right_leg_knee_link"/>
     <child link="right_leg_shin_link"/>
     <axis>
       <xyz>1 0 0</xyz>
-      <limit>
-          <lower>0</lower>
-          <upper>0</upper>
-      </limit>
     </axis>
     <origin xyz="0.015 -0.04 -0.09" rpy="0 0 0"/>

Commit message: Made changes to get full model working

File: hros1_description/urdf/hros1_body.xacro (robot description, xacro)
@@ -8,4 +8,5 @@
       <self_collide>0</self_collide>
       <kinematic>0</kinematic>
+      <static>1</static>
       <visual name='body_structure_visual'>
         <origin xyz="0 0 0"  rpy="0 -0 0"/>

File: hros1_description/urdf/hros1_right_leg.xacro (robot description, xacro)
@@ -61,5 +61,5 @@
         <origin xyz="0 0 0" rpy="0 -0 0"/>
         <geometry>
-          <mesh filename="model://HR-OS1/meshes/HROS1_Simple - Right_Leg_Thigh.stl"/>
+          <mesh filename="package://hros1_description/meshes/HROS1_Simple - Right_Leg_Thigh.stl"/>
         </geometry>
       </visual>
@@ -86,5 +86,5 @@
         <origin xyz="0 0 0" rpy="0 -0 0"/>
         <geometry>
-          <mesh filename="model://HR-OS1/meshes/HROS1_Simple - Right_Leg_Knee.stl"/>
+          <mesh filename="package://hros1_description/meshes/HROS1_Simple - Right_Leg_Knee.stl"/>
         </geometry>
       </visual>
@@ -167,7 +167,5 @@
         <origin xyz=" 0.05 -0.05 -0.195" rpy="0 0 0 "/>
         <geometry>
-          <box>
-            <size>0.065 .1 0.01</size>
-          </box>
+          <box size="0.065 .1 0.01"/>
         </geometry>
       </collision>
