Commit message: Got neck links working correctly

File: hros1_description/urdf/hros1_body.xacro (robot description, xacro)
@@ -9,4 +9,5 @@
       <kinematic>0</kinematic>
       <static>1</static>
+      <!--
       <visual name='body_structure_visual'>
         <origin xyz="0 0 0"  rpy="0 -0 0"/>
@@ -14,13 +15,6 @@
           <mesh filename="package://hros1_description/meshes/HROS1_Simple - Body_Structure.stl"/>
         </geometry>
-        <!--
-        <material>
-          <script>
-            <uri>file://media/materials/scripts/gazebo.material</uri>
-            <name>Gazebo/Grey</name>
-          </script>
-        </material>
-        -->
       </visual>
+      -->
       <collision name="collision">
         <origin xyz="0 -0.055 0.08" rpy="0 0 0"/>

File: hros1_description/urdf/hros1_left_arm.xacro (robot description, xacro)
@@ -53,4 +53,5 @@
     </link>
 <!--  LEFT ARM Elbow  -->
+<!--
     <link name='left_arm_elbow_link'>
       <origin xyz="0 0 0" rpy="0 -0 0"/>
@@ -77,5 +78,7 @@
       </inertial>
     </link>
+-->
 <!--  LEFT ARM FOREARM SERVO  -->
+<!--
     <link name='left_arm_forearm_servo_link'>
       <origin xyz="0 0 0" rpy="0 -0 0"/>
@@ -102,4 +105,5 @@
       </inertial>
     </link>
+    -->
 </xacro:macro>
 <xacro:macro name="left_arm_joints">

File: hros1_description/urdf/hros1_neck.xacro (robot description, xacro)
@@ -1,5 +1,31 @@
 <?xml version="1.0"?>
 <robot xmlns:xacro="http://ros.org/wiki/xacro">
-<!--  NECK Head (Pitch Servo) -->
+<xacro:macro name="neck_links">
+    <!--  ATTACHED TO TOP OF BODY -->
+    <link name='neck_link_1_link'>
+      <origin xyz="0 0 0" rpy="0 -0 0"/>
+      <gravity>1</gravity>
+      <self_collide>0</self_collide>
+      <kinematic>0</kinematic>
+      <visual name='neck_link_1_visual'>
+        <origin xyz="0 0 0" rpy="0 -0 0"/>
+        <geometry>
+          <mesh filename="package://hros1_description/meshes/hros1_neck_link_1_moved.stl"/>
+        </geometry>
+      </visual>
+      <inertial>
+        <origin xyz="0 -0.101 0.208" rpy="0 -0 0"/>
+        <mass value="0.005"/>
+        <inertia
+          ixx="0.0000012"
+          ixy="0.0"
+          ixz="0.0"
+          iyy="0.0000032"
+          iyz="0.0"
+          izz="0.000002"
+          />
+      </inertial>
+    </link>
+    <!--  NECK Head (Pitch Servo) -->
 <!--  ATTACHED TO BACK OF HEAD  -->
     <link name='neck_head_link'>
@@ -40,6 +66,5 @@
       <kinematic>0</kinematic>
       <visual name='neck_base_visual'>
-        <origin xyz="0 0 0" rpy="0 0 0"/>
-        <!--<origin xyz="0 0.052 0" rpy="0 -0 0"/>-->
+        <origin xyz="0 0 0" rpy="0 -0 3.1415"/>
         <geometry>
           <mesh filename="package://hros1_description/meshes/hros1_neck_base_moved.stl"/>
@@ -67,6 +92,5 @@
       <kinematic>0</kinematic>
       <visual name='neck_base_platform_visual'>
-        <origin xyz="0 0 0" rpy="0 0 0"/>
-        <!--<origin xyz="0 0.98 -.20" rpy="0 -0 0"/>-->
+        <origin xyz="0 0 0" rpy="0 -0 0"/>
         <geometry>
           <mesh filename="package://hros1_description/meshes/hros1_neck_base_platform_moved.stl"/>
@@ -106,5 +130,5 @@
       </visual>
       <inertial>
-        <origin xyz="0 -0.077 0.231" rpy="0 -0 0"/>
+        <origin xyz="0 0 0.046" rpy="0 -0 0"/>
         <mass value="0.011"/>
         <inertia
@@ -118,30 +142,4 @@
       </inertial>
     </link>
-<xacro:macro name="neck_links">
-    <!--  ATTACHED TO TOP OF BODY -->
-    <link name='neck_link_1_link'>
-      <origin xyz="0 0 0" rpy="0 -0 0"/>
-      <gravity>1</gravity>
-      <self_collide>0</self_collide>
-      <kinematic>0</kinematic>
-      <visual name='neck_link_1_visual'>
-        <origin xyz="0 0 0" rpy="0 -0 0"/>
-        <geometry>
-          <mesh filename="package://hros1_description/meshes/hros1_neck_link_1_moved.stl"/>
-        </geometry>
-      </visual>
-      <inertial>
-        <origin xyz="0 -0.101 0.208" rpy="0 -0 0"/>
-        <mass value="0.005"/>
-        <inertia
-          ixx="0.0000012"
-          ixy="0.0"
-          ixz="0.0"
-          iyy="0.0000032"
-          iyz="0.0"
-          izz="0.000002"
-          />
-      </inertial>
-    </link>
 </xacro:macro>
 <xacro:macro name="neck_joints">
@@ -150,8 +148,6 @@
     <child link="neck_base_link"/>
     <limit effort="1" velocity="1" lower="-3.1415" upper="3.1415"/>
-    <axis>
-      <xyz>0 0 1</xyz>
-    </axis>
-    <origin xyz="0 -0.052 0.162" rpy="0 0 3.1415"/>
+    <axis xyz="0 0 1"/>
+    <origin xyz="0 -0.052 0.162" rpy="0 0 0"/>
   </joint>
   <joint name="neck_base_platform_free_joint" type="continuous">
@@ -162,5 +158,5 @@
       <xyz>1 0 0</xyz>
     </axis>
-    <origin xyz="0 0 0.042" rpy="0 0 0"/>
+    <origin xyz="0.015 0 0.042" rpy="0 0 0"/>
   </joint>
   <joint name="neck_pitch_1_free_joint" type="continuous">
@@ -171,5 +167,5 @@
       <xyz>1 0 0</xyz>
     </axis>
-    <origin xyz="0 0.049 0.026" rpy="0 0 0"/>
+    <origin xyz="0 -0.049 0.028" rpy="0 0 0"/>
   </joint>
   <joint name="neck_pitch_2_free_joint" type="continuous">
@@ -180,5 +176,5 @@
       <xyz>1 0 0</xyz>
     </axis>
-    <origin xyz="0 0 0.048" rpy="0 0 0"/>
+    <origin xyz="0 0 0.048" rpy="0 0 3.1415"/>
   </joint>
   <joint name="neck_pitch_main_powered_joint" type="revolute">

File: hros1_description/urdf/hros1_robot.urdf.xacro (robot description, xacro)
@@ -4,7 +4,7 @@
     <xacro:include filename="$(find hros1_description)/urdf/hros1_body.xacro"/>
     <xacro:include filename="$(find hros1_description)/urdf/hros1_neck.xacro"/>
-<!--
     <xacro:include filename="$(find hros1_description)/urdf/hros1_left_arm.xacro"/>
     <xacro:include filename="$(find hros1_description)/urdf/hros1_left_leg.xacro"/>
+<!--
     <xacro:include filename="$(find hros1_description)/urdf/hros1_right_arm.xacro"/>
     <xacro:include filename="$(find hros1_description)/urdf/hros1_right_leg.xacro"/>
@@ -17,6 +17,10 @@
     <xacro:left_arm_links />
     <xacro:left_arm_joints />
+    -->
+    <!--
     <xacro:left_leg_links />
     <xacro:left_leg_joints />
+    -->
+    <!--
     <xacro:right_arm_links />
     <xacro:right_arm_joints />
@@ -24,3 +28,11 @@
     <xacro:right_leg_joints />
     -->
+    <link name="world"/>
+    <joint name="fixed_joint" type="fixed">
+        <parent link="world"/>
+        <child link="body_structure_link"/>
+        <axis>
+          <xyz>0 0 1</xyz>
+        </axis>
+    </joint>
 </robot>
