Commit message: Modified urdf files to be properly arranged

File: hros1_description/urdf/hros1_body.xacro (robot description, xacro)
@@ -9,12 +9,18 @@
       <kinematic>0</kinematic>
       <static>1</static>
-      <!--
       <visual name='body_structure_visual'>
         <origin xyz="0 0 0"  rpy="0 -0 0"/>
         <geometry>
-          <mesh filename="package://hros1_description/meshes/HROS1_Simple - Body_Structure.stl"/>
+          <mesh filename="package://hros1_description/meshes/body_structure.stl"/>
         </geometry>
+        <!--
+        <material>
+          <script>
+            <uri>file://media/materials/scripts/gazebo.material</uri>
+            <name>Gazebo/Grey</name>
+          </script>
+        </material>
+        -->
       </visual>
-      -->
       <collision name="collision">
         <origin xyz="0 -0.055 0.08" rpy="0 0 0"/>
@@ -46,5 +52,5 @@
         <pose>0 0 0 0 -0 0</pose>
         <geometry>
-          <mesh filename="package://hros1_description/meshes/HROS1_Simple - Body_Servos.stl"/>
+          <mesh filename="package://hros1_description/meshes/body_servos.stl"/>
         </geometry>
       </visual>
@@ -72,5 +78,5 @@
         <origin xyz="0 0 0" rpy="0 -0 0"/>
         <geometry>
-          <mesh filename="package://hros1_description/meshes/HROS1_Simple - Body_Battery.stl"/>
+          <mesh filename="package://hros1_description/meshes/body_battery.stl"/>
         </geometry>
       </visual>
@@ -90,5 +96,5 @@
 </xacro:macro>
 <xacro:macro name="body_joints">
-<joint name="body-servos_fixture_joint" type="fixed">
+<joint name="body_servos_fixture_joint" type="fixed">
     <parent link="body_structure_link"/>
     <child link="body_servos_link"/>
@@ -97,5 +103,5 @@
     </axis>
   </joint>
-  <joint name="body-battery_fixture_joint" type="fixed">
+  <joint name="body_battery_fixture_joint" type="fixed">
     <parent link="body_structure_link"/>
     <child link="body_battery_link"/>

File: hros1_description/urdf/hros1_left_arm.xacro (robot description, xacro)
@@ -1,144 +1,134 @@
 <?xml version="1.0"?>
 <robot xmlns:xacro="http://ros.org/wiki/xacro">
-<xacro:macro name="left_arm_links">
-<!--  LEFT ARM SHOULDER  -->
-    <link name='left_arm_shoulder_link'>
-      <origin xyz="0 0 0" rpy="0 -0 0"/>
-      <gravity>1</gravity>
-      <self_collide>0</self_collide>
-      <kinematic>0</kinematic>
-      <visual name='left_arm_shoulder_visual'>
-        <origin xyz="0 0 0" rpy="0 -0 0"/>
-        <geometry>
-          <mesh filename="package://hros1_description/meshes/HROS1_Simple - Left_Arm_Shoulder.stl"/>
-        </geometry>
-      </visual>
-      <inertial>
-        <origin xyz="0.068 -0.052 0.131" rpy="0 -0 0"/>
-        <mass value="0.011"/>
-        <inertia
-          ixx="0.0000051"
-          ixy="0.0"
-          ixz="0.00000058"
-          iyy="0.0000023"
-          iyz="0.0"
-          izz="0.000005"
-          />
-      </inertial>
-    </link>
-<!--  LEFT ARM UPPER SERVO  -->
-    <link name='left_arm_upper_servo_link'>
-      <origin xyz="0 0 0 0 -0 0"/>
-      <gravity>1</gravity>
-      <self_collide>0</self_collide>
-      <kinematic>0</kinematic>
-      <visual name='left_arm_upper_servo_visual'>
-        <origin xyz="0 0 0" rpy="0 -0 0"/>
-        <geometry>
-          <mesh filename="package://hros1_description/meshes/HROS1_Simple - Left_Arm_Upper_Servo.stl"/>
-        </geometry>
-      </visual>
-      <inertial>
-        <origin xyz="0.085 -0.051 0.106" rpy="0 -0 0"/>
-        <mass value="0.055"/>
-        <inertia
-          ixx="0.000015"
-          ixy="0.000000062"
-          ixz="0.0000017"
-          iyy="0.000013"
-          iyz="-0.00000025"
-          izz="0.0000089"
-          />
-      </inertial>
-    </link>
-<!--  LEFT ARM Elbow  -->
-<!--
-    <link name='left_arm_elbow_link'>
-      <origin xyz="0 0 0" rpy="0 -0 0"/>
-      <gravity>1</gravity>
-      <self_collide>0</self_collide>
-      <kinematic>0</kinematic>
-      <visual name='left_arm_elbow_visual'>
-        <origin xyz="0 0 0" rpy="0 -0 0"/>
-        <geometry>
-          <mesh filename="package://hros1_description/meshes/HROS1_Simple - Left_Arm_Elbow_Link.stl"/>
-        </geometry>
-      </visual>
-      <inertial>
-        <origin xyz="0.093 -0.050 0.072" rpy="0 -0 0"/>
-        <mass value="0.016"/>
-        <inertia
-          ixx="0.0000036"
-          ixy="0.00000016"
-          ixz="-0.00000062"
-          iyy="0.0000056"
-          iyz="-0.00000064"
-          izz="0.0000058"
-          />
-      </inertial>
-    </link>
--->
-<!--  LEFT ARM FOREARM SERVO  -->
-<!--
-    <link name='left_arm_forearm_servo_link'>
-      <origin xyz="0 0 0" rpy="0 -0 0"/>
-      <gravity>1</gravity>
-      <self_collide>0</self_collide>
-      <kinematic>0</kinematic>
-      <visual name='left_arm_forearm_servo_visual'>
-        <origin xyz="0 0 0" rpy="0 -0 0"/>
-        <geometry>
-          <mesh filename="package://hros1_description/meshes/HROS1_Simple - Left_Arm_Forearm_Servo.stl"/>
-        </geometry>
-      </visual>
-      <inertial>
-        <origin xyz="0.100 -0.028 0.047" rpy="0 -0 0"/>
-        <mass value="0.055"/>
-        <inertia
-          ixx="0.000013"
-          ixy="0.0000011"
-          ixz="0.00000051"
-          iyy="0.000012"
-          iyz="-0.0000034"
-          izz="0.000012"
-          />
-      </inertial>
-    </link>
-    -->
-</xacro:macro>
-<xacro:macro name="left_arm_joints">
-  <joint name="left_shoulder_pitch_powered_joint" type="revolute">
-    <parent link="body_structure_link"/>
-    <child link="left_arm_shoulder_link"/>
-    <axis>
-      <xyz>-1 0 0</xyz>
-    </axis>
-    <origin xyz="0 -0.05 0.13" rpy="0 0 0"/>
-    <limit effort="1" velocity="1" upper="3.1415" lower="-3.1415"/>
-  </joint>
-  <joint name="left_shoulder_roll_powered_joint" type="revolute">
-    <parent link="left_arm_shoulder_link"/>
-    <child link="left_arm_upper_servo_link"/>
-    <axis>
-      <xyz>0 -1 0</xyz>
-    </axis>
-    <origin xyz="-0.085 -0.05 0.115" rpy="0 0 0"/>
-    <limit effort="1" velocity="1" upper="3.1415" lower="-3.1415"/>
-  </joint>
-  <joint name="left_shoulder-elbow_fixed_joint" type="fixed">
-    <parent link="left_arm_upper_servo_link"/>
-    <child link="left_arm_elbow_link"/>
-    <axis>
-    </axis>
-  </joint>
-  <joint name="left_elbow_powered_joint" type="revolute">
-    <parent link="left_arm_elbow_link"/>
-    <child link="left_arm_forearm_servo_link"/>
-    <axis>
-      <xyz>1 0 -0.25</xyz>
-    </axis>
-    <origin xyz="0 -0.037 0.03" rpy="0 0 0"/>
-    <limit effort="1" velocity="1" upper="3.1415" lower="-3.1415"/>
-  </joint>
-</xacro:macro>
+    <xacro:macro name="left_arm_links">
+    <!--  LEFT ARM SHOULDER  -->
+        <link name='left_arm_shoulder_link'>
+          <origin xyz="0 0 0" rpy="0 -0 0"/>
+          <gravity>1</gravity>
+          <self_collide>0</self_collide>
+          <kinematic>0</kinematic>
+          <visual name='left_arm_shoulder_visual'>
+            <origin xyz="0 0 0" rpy="0 -0 0"/>
+            <geometry>
+              <mesh filename="package://hros1_description/meshes/hros1_left_arm_shoulder_moved.stl"/>
+            </geometry>
+          </visual>
+          <inertial>
+            <origin xyz="0.068 -0.052 0.131" rpy="0 -0 0"/>
+            <mass value="0.011"/>
+            <inertia
+              ixx="0.0000051"
+              ixy="0.0"
+              ixz="0.00000058"
+              iyy="0.0000023"
+              iyz="0.0"
+              izz="0.000005"
+              />
+          </inertial>
+        </link>
+    <!--  LEFT ARM UPPER SERVO  -->
+        <link name='left_arm_upper_servo_link'>
+          <origin xyz="0 0 0 0 -0 0"/>
+          <gravity>1</gravity>
+          <self_collide>0</self_collide>
+          <kinematic>0</kinematic>
+          <visual name='left_arm_upper_servo_visual'>
+            <origin xyz="0 0 0" rpy="0 -0 0"/>
+            <geometry>
+              <mesh filename="package://hros1_description/meshes/hros1_left_arm_upper_servo_moved.stl"/>
+            </geometry>
+          </visual>
+          <inertial>
+            <origin xyz="0.085 -0.051 0.106" rpy="0 -0 0"/>
+            <mass value="0.055"/>
+            <inertia
+              ixx="0.000015"
+              ixy="0.000000062"
+              ixz="0.0000017"
+              iyy="0.000013"
+              iyz="-0.00000025"
+              izz="0.0000089"
+              />
+          </inertial>
+        </link>
+    <!--  LEFT ARM Elbow  -->
+        <link name='left_arm_elbow_link'>
+          <origin xyz="0 0 0" rpy="0 -0 0"/>
+          <gravity>1</gravity>
+          <self_collide>0</self_collide>
+          <kinematic>0</kinematic>
+          <visual name='left_arm_elbow_visual'>
+            <origin xyz="0 0 0" rpy="0 -0 0"/>
+            <geometry>
+              <mesh filename="package://hros1_description/meshes/hros1_left_arm_elbow_link_moved.stl"/>
+            </geometry>
+          </visual>
+          <inertial>
+            <origin xyz="0.093 -0.050 0.072" rpy="0 -0 0"/>
+            <mass value="0.016"/>
+            <inertia
+              ixx="0.0000036"
+              ixy="0.00000016"
+              ixz="-0.00000062"
+              iyy="0.0000056"
+              iyz="-0.00000064"
+              izz="0.0000058"
+              />
+          </inertial>
+        </link>
+    <!--  LEFT ARM FOREARM SERVO  -->
+        <link name='left_arm_forearm_servo_link'>
+          <origin xyz="0 0 0" rpy="0 -0 0"/>
+          <gravity>1</gravity>
+          <self_collide>0</self_collide>
+          <kinematic>0</kinematic>
+          <visual name='left_arm_forearm_servo_visual'>
+            <origin xyz="0 0 0" rpy="0 -0 0"/>
+            <geometry>
+              <mesh filename="package://hros1_description/meshes/hros1_left_arm_forearm_servo_moved.stl"/>
+            </geometry>
+          </visual>
+          <inertial>
+            <origin xyz="0.100 -0.028 0.047" rpy="0 -0 0"/>
+            <mass value="0.055"/>
+            <inertia
+              ixx="0.000013"
+              ixy="0.0000011"
+              ixz="0.00000051"
+              iyy="0.000012"
+              iyz="-0.0000034"
+              izz="0.000012"
+              />
+          </inertial>
+        </link>
+    </xacro:macro>
+    <xacro:macro name="left_arm_joints">
+      <joint name="left_shoulder_pitch_powered_joint" type="revolute">
+        <parent link="body_structure_link"/>
+        <child link="left_arm_shoulder_link"/>
+        <axis xyz="-1 0 0"/>
+        <origin xyz="0.051 0.052 0.133" rpy="0 0 0"/>
+        <limit effort="1" velocity="1" upper="3.1415" lower="-3.1415"/>
+      </joint>
+      <joint name="left_shoulder_roll_powered_joint" type="revolute">
+        <parent link="left_arm_shoulder_link"/>
+        <child link="left_arm_upper_servo_link"/>
+        <axis xyz="0 -1 0"/>
+        <origin xyz="0.03 0.02 -0.015" rpy="0 0 0"/>
+        <limit effort="1" velocity="1" upper="3.1415" lower="-3.1415"/>
+      </joint>
+      <joint name="left_shoulder-elbow_fixed_joint" type="fixed">
+        <parent link="left_arm_upper_servo_link"/>
+        <child link="left_arm_elbow_link"/>
+        <axis xyz="0 -1 0"/>
+        <origin xyz="0.002 -0.033 -0.037" rpy="0 0 0"/>
+      </joint>
+      <joint name="left_elbow_powered_joint" type="revolute">
+        <parent link="left_arm_elbow_link"/>
+        <child link="left_arm_forearm_servo_link"/>
+        <axis xyz="-0.8 0.0 -0.2"/>
+        <origin xyz="-0.005 0.0 -0.03" rpy="0 0 0"/>
+        <limit effort="1" velocity="1" upper="3.1415" lower="-3.1415"/>
+      </joint>
+    </xacro:macro>
 </robot>

File: hros1_description/urdf/hros1_left_leg.xacro (robot description, xacro)
@@ -28,4 +28,5 @@
     </link>
 <!-- LEFT LOWER HIP  -->
+<!--
     <link name='left_leg_lower_hip_link'>
       <origin xyz="0 0 0 0 -0 0"/>
@@ -52,5 +53,7 @@
       </inertial>
     </link>
+-->
 <!-- LEFT THIGH  -->
+<!--
     <link name='left_leg_thigh_link'>
       <origin xyz="0 0 0 0 -0 0"/>
@@ -77,5 +80,7 @@
       </inertial>
     </link>
+-->
 <!-- LEFT KNEE  -->
+<!--
     <link name='left_leg_knee_link'>
       <origin xyz="0 0 0" rpy="0 -0 0"/>
@@ -102,5 +107,7 @@
       </inertial>
     </link>
+-->
 <!-- LEFT SHIN  -->
+<!--
     <link name='left_leg_shin_link'>
       <origin xyz="0 0 0" rpy="0 -0 0"/>
@@ -127,5 +134,7 @@
       </inertial>
     </link>
+-->
 <!-- LEFT ANKLE  -->
+<!--
     <link name='left_leg_ankle_link'>
       <origin xyz="0 0 0" rpy="0 -0 0"/>
@@ -152,5 +161,7 @@
       </inertial>
     </link>
+-->
 <!-- LEFT FOOT  -->
+<!--
     <link name='left_leg_foot_link'>
       <origin xyz="0 0 0" rpy="0 -0 0"/>
@@ -183,4 +194,5 @@
       </inertial>
     </link>
+ -->
 </xacro:macro>
 <xacro:macro name="left_leg_joints">
@@ -188,16 +200,13 @@
     <parent link="body_structure_link"/>
     <child link="left_leg_upper_hip_link"/>
-    <axis>
-      <xyz>0 0 -1</xyz>
-    </axis>
+    <axis xyz="0 0 1"/>
     <origin xyz="-0.040 -0.045 0" rpy="0 0 0"/>
     <limit effort="1" velocity="1" upper="3.1415" lower="-3.1415"/>
   </joint>
+  <!--
   <joint name="left_hip_roll_powered_joint" type="revolute">
     <parent link="left_leg_upper_hip_link"/>
     <child link="left_leg_lower_hip_link"/>
-    <axis>
-      <xyz>0 1 0</xyz>
-    </axis>
+    <axis xyz="0 0 1"/>
     <origin xyz="-0.040 -0.045 -0.01" rpy="0 0 0"/>
     <limit effort="1" velocity="1" upper="3.1415" lower="-3.1415"/>
@@ -206,7 +215,5 @@
     <parent link="left_leg_lower_hip_link"/>
     <child link="left_leg_thigh_link"/>
-    <axis>
-      <xyz>1 0 0</xyz>
-    </axis>
+    <axis xyz="0 0 1"/>
     <origin xyz="-0.040 -0.045 -0.01" rpy="0 0 0"/>
     <limit effort="1" velocity="1" upper="3.1415" lower="-3.1415"/>
@@ -215,7 +222,5 @@
     <parent link="left_leg_thigh_link"/>
     <child link="left_leg_knee_link"/>
-    <axis>
-      <xyz>-1 0 0</xyz>
-    </axis>
+    <axis xyz="0 0 1"/>
     <origin xyz="-0.015 -0.04 -0.09" rpy="0 0 0"/>
     <limit effort="1" velocity="1" upper="3.1415" lower="-3.1415"/>
@@ -224,7 +229,5 @@
     <parent link="left_leg_knee_link"/>
     <child link="left_leg_shin_link"/>
-    <axis>
-      <xyz>1 0 0</xyz>
-    </axis>
+    <axis xyz="0 0 1"/>
     <origin xyz="-0.015 -0.04 -0.09" rpy="0 0 0"/>
     <limit effort="1" velocity="1" upper="3.1415" lower="-3.1415"/>
@@ -233,7 +236,5 @@
     <parent link="left_leg_shin_link"/>
     <child link="left_leg_ankle_link"/>
-    <axis>
-      <xyz>-1 0 0</xyz>
-    </axis>
+    <axis xyz="0 0 1"/>
     <origin xyz="-0.015 -0.045 -0.16" rpy="0 0 0"/>
     <limit effort="1" velocity="1" upper="3.1415" lower="-3.1415"/>
@@ -242,10 +243,9 @@
     <parent link="left_leg_ankle_link"/>
     <child link="left_leg_foot_link"/>
-    <axis>
-      <xyz>0 -1 0</xyz>
-    </axis>
+    <axis xyz="0 0 1"/>
     <origin xyz="-0.04 -0.045 -0.16" rpy="0 0 0"/>
     <limit effort="1" velocity="1" upper="3.1415" lower="-3.1415"/>
   </joint>
+  -->
 </xacro:macro>
 </robot>

File: hros1_description/urdf/hros1_neck.xacro (robot description, xacro)
@@ -61,10 +61,10 @@
 <!--  ATTACHED TO BACK OF HEAD  -->
     <link name='neck_base_link'>
-      <!--<origin xyz="0 0.18 0.188" rpy="0 -0 0"/>-->
+      <origin xyz="0 0.0 0.0" rpy="0 -0 0"/>
       <gravity>1</gravity>
       <self_collide>0</self_collide>
       <kinematic>0</kinematic>
       <visual name='neck_base_visual'>
-        <origin xyz="0 0 0" rpy="0 -0 3.1415"/>
+        <origin xyz="0 0.0 0" rpy="0 -0 0"/>
         <geometry>
           <mesh filename="package://hros1_description/meshes/hros1_neck_base_moved.stl"/>
@@ -130,5 +130,5 @@
       </visual>
       <inertial>
-        <origin xyz="0 0 0.046" rpy="0 -0 0"/>
+        <origin xyz="0 -0.077 0.231" rpy="0 -0 0"/>
         <mass value="0.011"/>
         <inertia
@@ -149,14 +149,12 @@
     <limit effort="1" velocity="1" lower="-3.1415" upper="3.1415"/>
     <axis xyz="0 0 1"/>
-    <origin xyz="0 -0.052 0.162" rpy="0 0 0"/>
+    <origin xyz="0 0.052 0.16" rpy="0 -0 0"/>
   </joint>
-  <joint name="neck_base_platform_free_joint" type="continuous">
+  <joint name="neck_base_platform_free_joint" type="revolute">
     <parent link="neck_base_link"/>
     <child link="neck_base_platform_link"/>
     <limit effort="0" velocity="1" upper="3.1415" lower="-3.1415"/>
-    <axis>
-      <xyz>1 0 0</xyz>
-    </axis>
-    <origin xyz="0.015 0 0.042" rpy="0 0 0"/>
+    <axis xyz="1 0 0"/>
+    <origin xyz="0.0 0.0005 0.0425" rpy="0 -0 0"/>
   </joint>
   <joint name="neck_pitch_1_free_joint" type="continuous">
@@ -164,8 +162,6 @@
     <child link="neck_link_1_link"/>
     <limit effort="0" velocity="1" upper="3.1415" lower="-3.1415"/>
-    <axis>
-      <xyz>1 0 0</xyz>
-    </axis>
-    <origin xyz="0 -0.049 0.028" rpy="0 0 0"/>
+    <axis xyz="1 0 0"/>
+    <origin xyz="0 0.05 0.026" rpy="0 -0 0"/>
   </joint>
   <joint name="neck_pitch_2_free_joint" type="continuous">
@@ -173,8 +169,6 @@
     <child link="neck_link_2_link"/>
     <limit effort="0" velocity="1" upper="3.1415" lower="-3.1415"/>
-    <axis>
-      <xyz>1 0 0</xyz>
-    </axis>
-    <origin xyz="0 0 0.048" rpy="0 0 3.1415"/>
+    <axis xyz="1 0 0"/>
+    <origin xyz="0 0 0.046" rpy="0 -0 0"/>
   </joint>
   <joint name="neck_pitch_main_powered_joint" type="revolute">
@@ -182,8 +176,6 @@
     <child link="neck_head_link"/>
     <limit effort="1" velocity="1" upper="3.1415" lower="-3.1415"/>
-    <axis>
-      <xyz>-1 0 0</xyz>
-    </axis>
-    <origin xyz="0 -0.034 0.0" rpy="0 0 0"/>
+    <axis xyz="-1 0 0"/>
+    <origin xyz="0 -0.034 0.0" rpy="0 -0 0"/>
   </joint>
 </xacro:macro>

File: hros1_description/urdf/hros1_robot.urdf.xacro (robot description, xacro)
@@ -14,12 +14,8 @@
     <xacro:neck_links />
     <xacro:neck_joints />
-    <!--
     <xacro:left_arm_links />
     <xacro:left_arm_joints />
-    -->
-    <!--
     <xacro:left_leg_links />
     <xacro:left_leg_joints />
-    -->
     <!--
     <xacro:right_arm_links />
