Commit message: Changed/checked mass, inertial, and CoM values based on CAD files

File: hros1_description/urdf/hros1_body.xacro (robot description, xacro)
@@ -30,5 +30,5 @@
       </collision>
       <inertial>
-        <origin xyz="0 -0.065 0.082" rpy=" 0 -0 0"/>
+        <origin xyz="0 0.065 0.082" rpy=" 0 -0 0"/>
         <mass value="0.273"/>
         <inertia
@@ -56,5 +56,5 @@
       </visual>
       <inertial>
-        <origin xyz="0 -0.055 0.086" rpy=" 0 -0 0"/>
+        <origin xyz="0 0.055 0.086" rpy=" 0 -0 0"/>
         <mass value="0.221"/>
         <inertia
@@ -82,5 +82,5 @@
       </visual>
       <inertial>
-        <origin xyz="0 -0.078 0.036" rpy=" 0 -0 0"/>
+        <origin xyz="0 0.078 0.036" rpy=" 0 -0 0"/>
         <mass value="0.25"/>
         <inertia

File: hros1_description/urdf/hros1_left_arm.xacro (robot description, xacro)
@@ -15,5 +15,5 @@
           </visual>
           <inertial>
-            <origin xyz="0.068 -0.052 0.131" rpy="0 -0 0"/>
+            <origin xyz="0.016 0 -0.002" rpy="0 -0 0"/>
             <mass value="0.011"/>
             <inertia
@@ -40,5 +40,5 @@
           </visual>
           <inertial>
-            <origin xyz="0.085 -0.051 0.106" rpy="0 -0 0"/>
+            <origin xyz="0.004 -0.019 -0.013" rpy="0 -0 0"/>
             <mass value="0.055"/>
             <inertia
@@ -65,5 +65,5 @@
           </visual>
           <inertial>
-            <origin xyz="0.093 -0.050 0.072" rpy="0 -0 0"/>
+            <origin xyz="0.011 0.014 -0.009" rpy="0 -0 0"/>
             <mass value="0.016"/>
             <inertia
@@ -90,5 +90,5 @@
           </visual>
           <inertial>
-            <origin xyz="0.100 -0.028 0.047" rpy="0 -0 0"/>
+            <origin xyz="0.021 -0.010 -0.004" rpy="0 -0 0"/>
             <mass value="0.055"/>
             <inertia

File: hros1_description/urdf/hros1_left_leg.xacro (robot description, xacro)
@@ -15,5 +15,5 @@
       </visual>
       <inertial>
-        <origin xyz="0.039 -0.062 0.011" rpy="0 -0 0"/>
+        <origin xyz="0 0.017 -0.014" rpy="0 -0 0"/>
         <mass value="0.017"/>
         <inertia
@@ -40,5 +40,5 @@
       </visual>
       <inertial>
-        <origin xyz="0.039 -0.062 -0.024" rpy="0 -0 0"/>
+        <origin xyz="0.0 -0.037 -0.013" rpy="0 -0 0"/>
         <mass value="0.110"/>
         <inertia
@@ -65,5 +65,5 @@
       </visual>
       <inertial>
-        <origin xyz="0.039 -0.034 -0.053" rpy="0 -0 0"/>
+        <origin xyz="0.015 -0.011 -0.043" rpy="0 -0 0"/>
         <mass value="0.028"/>
         <inertia
@@ -90,5 +90,5 @@
       </visual>
       <inertial>
-        <origin xyz="0.038 -0.027 -0.091" rpy="0 -0 0"/>
+        <origin xyz="0.020 -0.013 -0.004" rpy="0 -0 0"/>
         <mass value="0.055"/>
         <inertia
@@ -115,5 +115,5 @@
       </visual>
       <inertial>
-        <origin xyz="0.039 -0.035 -0.125" rpy="0 -0 0"/>
+        <origin xyz="0.017 -0.002 -0.023" rpy="0 -0 0"/>
         <mass value="0.021"/>
         <inertia
@@ -140,5 +140,5 @@
       </visual>
       <inertial>
-        <origin xyz="0.039 -0.062 -0.147" rpy="0 -0 0"/>
+        <origin xyz="0.020 0.016 0.013" rpy="0 -0 0"/>
         <mass value="0.110"/>
         <inertia
@@ -171,5 +171,5 @@
       </collision>
       <inertial>
-        <origin xyz="0.046 -0.052 -0.188" rpy="0 -0 0"/>
+        <origin xyz="0.008 -0.046 -0.028" rpy="0 -0 0"/>
         <mass value="0.067"/>
         <inertia

File: hros1_description/urdf/hros1_neck.xacro (robot description, xacro)
@@ -15,5 +15,5 @@
       </visual>
       <inertial>
-        <origin xyz="0 -0.101 0.208" rpy="0 -0 0"/>
+        <origin xyz="0 0 0.023" rpy="0 -0 0"/>
         <mass value="0.005"/>
         <inertia
@@ -47,4 +47,5 @@
       </collision>
       <inertial>
+        <origin xyz="0 -0.015 -0.005" rpy="0 -0 0"/>
         <mass value="0.127"/>
         <inertia
@@ -72,5 +73,5 @@
       </visual>
       <inertial>
-        <origin xyz="0 0.052 0" rpy="0 -0 0"/>
+        <origin xyz="0 0.017 0.02" rpy="0 -0 0"/>
         <mass value="0.075"/>
         <inertia
@@ -104,5 +105,5 @@
       </collision>
       <inertial>
-        <origin xyz="0 -0.052 0.207" rpy="0 -0 0"/>
+        <origin xyz="0 0 0.006" rpy="0 -0 0"/>
         <mass value="0.012"/>
         <inertia
@@ -130,5 +131,5 @@
       </visual>
       <inertial>
-        <origin xyz="0 -0.077 0.231" rpy="0 -0 0"/>
+        <origin xyz="0.001 -0.024 0.0" rpy="0 -0 0"/>
         <mass value="0.011"/>
         <inertia

File: hros1_description/urdf/hros1_right_arm.xacro (robot description, xacro)
@@ -14,5 +14,5 @@
       </visual>
       <inertial>
-        <origin xyz="-0.068 -0.052 0.131" rpy="0 -0 0"/>
+        <origin xyz="-0.016 0 -0.002" rpy="0 -0 0"/>
         <mass value="0.011"/>
         <inertia
@@ -39,5 +39,5 @@
       </visual>
       <inertial>
-        <origin xyz="-0.085 -0.051 0.106" rpy="0 -0 0"/>
+        <origin xyz="-0.003 -0.019 -0.013" rpy="0 -0 0"/>
         <mass value="0.055"/>
         <inertia
@@ -64,5 +64,5 @@
       </visual>
       <inertial>
-        <origin xyz="-0.093 -0.050 0.072" rpy="0 -0 0"/>
+        <origin xyz="-0.011 0.015 -0.010" rpy="0 -0 0"/>
         <mass value="0.016"/>
         <inertia
@@ -89,5 +89,5 @@
       </visual>
       <inertial>
-        <origin xyz="-0.100 -0.028 0.047" rpy="0 -0 0"/>
+        <origin xyz="-0.021 -0.009 -0.004" rpy="0 -0 0"/>
         <mass value="0.055"/>
         <inertia

File: hros1_description/urdf/hros1_right_leg.xacro (robot description, xacro)
@@ -15,5 +15,5 @@
       </visual>
       <inertial>
-        <origin xyz="-0.039 -0.062 0.011" rpy="0 -0 0"/>
+        <origin xyz="0 0.017 -0.014" rpy="0 -0 0"/>
         <mass value="0.017"/>
         <inertia
@@ -40,5 +40,5 @@
       </visual>
       <inertial>
-        <origin xyz="-0.039 -0.062 -0.024" rpy="0 -0 0"/>
+        <origin xyz="0 -0.037 -0.013" rpy="0 -0 0"/>
         <mass value="0.110"/>
         <inertia
@@ -65,5 +65,5 @@
       </visual>
       <inertial>
-        <origin xyz="-0.039 -0.034 -0.053" rpy="0 -0 0"/>
+        <origin xyz="-0.014 -0.011 -0.043" rpy="0 -0 0"/>
         <mass value="0.028"/>
         <inertia
@@ -90,5 +90,5 @@
       </visual>
       <inertial>
-        <origin xyz="-0.038 -0.027 -0.091" rpy="0 -0 0"/>
+        <origin xyz="-0.021 -0.013 -0.004" rpy="0 -0 0"/>
         <mass value="0.055"/>
         <inertia
@@ -115,5 +115,5 @@
       </visual>
       <inertial>
-        <origin xyz="-0.039 -0.035 -0.125" rpy="0 -0 0"/>
+        <origin xyz="-0.016 -0.002 -0.023" rpy="0 -0 0"/>
         <mass value="0.021"/>
         <inertia
@@ -140,5 +140,5 @@
       </visual>
       <inertial>
-        <origin xyz="-0.039 -0.062 -0.147" rpy="0 -0 0"/>
+        <origin xyz="-0.021 0.016 0.013" rpy="0 -0 0"/>
         <mass value="0.110"/>
         <inertia
@@ -171,5 +171,5 @@
       </collision>
       <inertial>
-        <origin xyz="-0.046 -0.052 -0.188" rpy="0 -0 0"/>
+        <origin xyz="-0.008 -0.045 -0.028" rpy="0 -0 0"/>
         <mass value="0.067"/>
         <inertia

Commit message: Made body dynamic

File: hros1_description/urdf/hros1_body.xacro (robot description, xacro)
@@ -8,5 +8,5 @@
       <self_collide>0</self_collide>
       <kinematic>0</kinematic>
-      <static>1</static>
+      <static>0</static>
       <visual name='body_structure_visual'>
         <origin xyz="0 0 0"  rpy="0 -0 0"/>

File: hros1_description/urdf/hros1_robot.urdf.xacro (robot description, xacro)
@@ -21,5 +21,5 @@
     <xacro:right_leg_joints />
     <link name="world"/>
-    <joint name="fixed_joint" type="fixed">
+    <joint name="fixed_joint" type="free">
         <parent link="world"/>
         <child link="body_structure_link"/>

Commit message: Created basic control package; Needs tuning

File: hros1_description/urdf/hros1_body.xacro (robot description, xacro)
@@ -24,5 +24,5 @@
       </visual>
       <collision name="collision">
-        <origin xyz="0 -0.055 0.08" rpy="0 0 0"/>
+        <origin xyz="0 0.055 0.08" rpy="0 0 0"/>
         <geometry>
           <box size="0.08 0.07 0.12"/>

File: hros1_description/urdf/hros1_left_arm.xacro (robot description, xacro)
@@ -109,5 +109,5 @@
         <axis xyz="-1 0 0"/>
         <origin xyz="0.051 0.052 0.133" rpy="0 0 0"/>
-        <limit effort="1" velocity="1" upper="3.1415" lower="-3.1415"/>
+        <xacro:ax12_limits />
       </joint>
       <joint name="left_shoulder_roll_powered_joint" type="revolute">
@@ -116,5 +116,5 @@
         <axis xyz="0 -1 0"/>
         <origin xyz="0.03 0.02 -0.015" rpy="0 0 0"/>
-        <limit effort="1" velocity="1" upper="3.1415" lower="-3.1415"/>
+        <xacro:ax12_limits />
       </joint>
       <joint name="left_shoulder-elbow_fixed_joint" type="fixed">
@@ -129,5 +129,5 @@
         <axis xyz="-0.8 0.0 -0.2"/>
         <origin xyz="-0.005 0.0 -0.03" rpy="0 0 0"/>
-        <limit effort="1" velocity="1" upper="3.1415" lower="-3.1415"/>
+        <xacro:ax12_limits />
       </joint>
     </xacro:macro>

File: hros1_description/urdf/hros1_left_leg.xacro (robot description, xacro)
@@ -191,5 +191,5 @@
     <axis xyz="0 0 1"/>
     <origin xyz="0.039 0.045 0.023" rpy="0 0 0"/>
-    <limit effort="1" velocity="1" upper="3.1415" lower="-3.1415"/>
+    <xacro:ax12_limits />
   </joint>
   <joint name="left_hip_roll_powered_joint" type="revolute">
@@ -198,5 +198,5 @@
     <axis xyz="0 1 0"/>
     <origin xyz="0 0.053 -0.036" rpy="0 0 0"/>
-    <limit effort="1" velocity="1" upper="3.1415" lower="-3.1415"/>
+    <xacro:ax12_limits />
   </joint>
   <joint name="left_hip_pitch_powered_joint" type="revolute">
@@ -205,5 +205,5 @@
     <axis xyz="1 0 0"/>
     <origin xyz="-0.015 -0.053 0" rpy="0 0 0"/>
-    <limit effort="1" velocity="1" upper="3.1415" lower="-3.1415"/>
+    <xacro:ax12_limits />
   </joint>
   <joint name="left_knee_pitch_powered_joint" type="revolute">
@@ -212,5 +212,5 @@
     <axis xyz="1 0 0"/>
     <origin xyz="-0.006 -0.006 -0.077" rpy="0 0 0"/>
-    <limit effort="1" velocity="1" upper="3.1415" lower="-3.1415"/>
+    <xacro:ax12_limits />
   </joint>
   <joint name="left_knee-shin_fixed_joint" type="fixed">
@@ -219,5 +219,5 @@
     <axis xyz="0 0 1"/>
     <origin xyz="0.004 -0.002 -0.015" rpy="0 0 0"/>
-    <limit effort="1" velocity="1" upper="3.1415" lower="-3.1415"/>
+    <xacro:ax12_limits />
   </joint>
   <joint name="left_ankle_pitch_powered_joint" type="revolute">
@@ -226,5 +226,5 @@
     <axis xyz="1 0 0"/>
     <origin xyz="-0.004 0.008 -0.058" rpy="0 0 0"/>
-    <limit effort="1" velocity="1" upper="3.1415" lower="-3.1415"/>
+    <xacro:ax12_limits />
   </joint>
   <joint name="left_ankle_roll_powered_joint" type="revolute">
@@ -233,5 +233,5 @@
     <axis xyz="0 1 0"/>
     <origin xyz="0.021 0.053 0" rpy="0 0 0"/>
-    <limit effort="1" velocity="1" upper="3.1415" lower="-3.1415"/>
+    <xacro:ax12_limits />
   </joint>
 </xacro:macro>

File: hros1_description/urdf/hros1_neck.xacro (robot description, xacro)
@@ -148,5 +148,6 @@
     <parent link="body_structure_link"/>
     <child link="neck_base_link"/>
-    <limit effort="1" velocity="1" lower="-3.1415" upper="3.1415"/>
+    <xacro:ax12_limits />
+    <xacro:ax12_dynamics />
     <axis xyz="0 0 1"/>
     <origin xyz="0 0.052 0.16" rpy="0 -0 0"/>
@@ -156,4 +157,5 @@
     <child link="neck_base_platform_link"/>
     <limit effort="0" velocity="1" upper="3.1415" lower="-3.1415"/>
+    <xacro:loose_dynamics />
     <axis xyz="1 0 0"/>
     <origin xyz="0.0 0.0005 0.0425" rpy="0 -0 0"/>
@@ -163,4 +165,5 @@
     <child link="neck_link_1_link"/>
     <limit effort="0" velocity="1" upper="3.1415" lower="-3.1415"/>
+    <xacro:loose_dynamics />
     <axis xyz="1 0 0"/>
     <origin xyz="0 0.05 0.026" rpy="0 -0 0"/>
@@ -170,4 +173,5 @@
     <child link="neck_link_2_link"/>
     <limit effort="0" velocity="1" upper="3.1415" lower="-3.1415"/>
+    <xacro:loose_dynamics />
     <axis xyz="1 0 0"/>
     <origin xyz="0 0 0.046" rpy="0 -0 0"/>
@@ -176,5 +180,6 @@
     <parent link="neck_link_2_link"/>
     <child link="neck_head_link"/>
-    <limit effort="1" velocity="1" upper="3.1415" lower="-3.1415"/>
+    <xacro:ax12_limits />
+    <xacro:ax12_dynamics />
     <axis xyz="-1 0 0"/>
     <origin xyz="0 -0.034 0.0" rpy="0 -0 0"/>

File: hros1_description/urdf/hros1_right_arm.xacro (robot description, xacro)
@@ -108,5 +108,5 @@
     <axis xyz="-1 0 0"/>
     <origin xyz="-0.051 0.052 0.133" rpy="0 0 0"/>
-    <limit effort="1" velocity="1" upper="3.1415" lower="-3.1415"/>
+    <xacro:ax12_limits />
   </joint>
   <joint name="right_shoulder_roll_powered_joint" type="revolute">
@@ -115,5 +115,5 @@
     <axis xyz="0 -1 0"/>
     <origin xyz="-0.03 0.02 -0.015" rpy="0 0 0"/>
-    <limit effort="1" velocity="1" upper="3.1415" lower="-3.1415"/>
+    <xacro:ax12_limits />
   </joint>
   <joint name="right_shoulder-elbow_fixed_joint" type="fixed">
@@ -128,5 +128,5 @@
     <axis xyz="-0.8 0.0 0.2"/>
     <origin xyz="0.005 0.0 -0.03" rpy="0 0 0"/>
-    <limit effort="1" velocity="1" upper="3.1415" lower="-3.1415"/>
+    <xacro:ax12_limits />
   </joint>
 </xacro:macro>

File: hros1_description/urdf/hros1_right_leg.xacro (robot description, xacro)
@@ -190,5 +190,5 @@
     <axis xyz="0 0 1"/>
     <origin xyz="-0.039 0.045 0.023" rpy="0 0 0"/>
-    <limit effort="1" velocity="1" upper="3.1415" lower="-3.1415"/>
+    <xacro:ax12_limits />
   </joint>
   <joint name="right_hip_roll_powered_joint" type="revolute">
@@ -197,5 +197,5 @@
     <axis xyz="0 1 0"/>
     <origin xyz="-0 0.053 -0.036" rpy="0 0 0"/>
-    <limit effort="1" velocity="1" upper="3.1415" lower="-3.1415"/>
+    <xacro:ax12_limits />
   </joint>
   <joint name="right_hip_pitch_powered_joint" type="revolute">
@@ -204,5 +204,5 @@
     <axis xyz="1 0 0"/>
     <origin xyz="0.015 -0.053 0" rpy="0 0 0"/>
-    <limit effort="1" velocity="1" upper="3.1415" lower="-3.1415"/>
+    <xacro:ax12_limits />
   </joint>
   <joint name="right_knee_pitch_powered_joint" type="revolute">
@@ -211,5 +211,5 @@
     <axis xyz="1 0 0"/>
     <origin xyz="0.006 -0.006 -0.077" rpy="0 0 0"/>
-    <limit effort="1" velocity="1" upper="3.1415" lower="-3.1415"/>
+    <xacro:ax12_limits />
   </joint>
   <joint name="right_knee-shin_fixed_joint" type="fixed">
@@ -225,5 +225,5 @@
     <axis xyz="1 0 0"/>
     <origin xyz="0.004 0.008 -0.058" rpy="0 0 0"/>
-    <limit effort="1" velocity="1" upper="3.1415" lower="-3.1415"/>
+    <xacro:ax12_limits />
   </joint>
   <joint name="right_ankle_roll_powered_joint" type="revolute">
@@ -232,5 +232,5 @@
     <axis xyz="0 1 0"/>
     <origin xyz="-0.021 0.053 0" rpy="0 0 0"/>
-    <limit effort="1" velocity="1" upper="3.1415" lower="-3.1415"/>
+    <xacro:ax12_limits />
   </joint>
 </xacro:macro>

File: hros1_description/urdf/hros1_robot.urdf (robot description, URDF)
Before this commit: robot hros1, 31 links, 30 joints
Joints:
- joint fixed_joint: type fixed -> floating
- joint left_ankle_pitch_powered_joint: limit lower=-3.1415 upper=3.1415 effort=1 velocity=1 -> lower=-3.1415 upper=3.1415 effort=1.5 velocity=59
- joint left_ankle_roll_powered_joint: limit lower=-3.1415 upper=3.1415 effort=1 velocity=1 -> lower=-3.1415 upper=3.1415 effort=1.5 velocity=59
- joint left_elbow_powered_joint: limit lower=-3.1415 upper=3.1415 effort=1 velocity=1 -> lower=-3.1415 upper=3.1415 effort=1.5 velocity=59
- joint left_hip_pitch_powered_joint: limit lower=-3.1415 upper=3.1415 effort=1 velocity=1 -> lower=-3.1415 upper=3.1415 effort=1.5 velocity=59
- joint left_hip_roll_powered_joint: limit lower=-3.1415 upper=3.1415 effort=1 velocity=1 -> lower=-3.1415 upper=3.1415 effort=1.5 velocity=59
- joint left_hip_yaw_powered_joint: limit lower=-3.1415 upper=3.1415 effort=1 velocity=1 -> lower=-3.1415 upper=3.1415 effort=1.5 velocity=59
- joint left_knee-shin_fixed_joint: limit lower=-3.1415 upper=3.1415 effort=1 velocity=1 -> lower=-3.1415 upper=3.1415 effort=1.5 velocity=59
- joint left_knee_pitch_powered_joint: limit lower=-3.1415 upper=3.1415 effort=1 velocity=1 -> lower=-3.1415 upper=3.1415 effort=1.5 velocity=59
- joint left_shoulder_pitch_powered_joint: limit lower=-3.1415 upper=3.1415 effort=1 velocity=1 -> lower=-3.1415 upper=3.1415 effort=1.5 velocity=59
- joint left_shoulder_roll_powered_joint: limit lower=-3.1415 upper=3.1415 effort=1 velocity=1 -> lower=-3.1415 upper=3.1415 effort=1.5 velocity=59
- joint neck_pitch_main_powered_joint: limit lower=-3.1415 upper=3.1415 effort=1 velocity=1 -> lower=-3.1415 upper=3.1415 effort=1.5 velocity=59
- joint neck_yaw_powered_joint: limit lower=-3.1415 upper=3.1415 effort=1 velocity=1 -> lower=-3.1415 upper=3.1415 effort=1.5 velocity=59
- joint right_ankle_pitch_powered_joint: limit lower=-3.1415 upper=3.1415 effort=1 velocity=1 -> lower=-3.1415 upper=3.1415 effort=1.5 velocity=59
- joint right_ankle_roll_powered_joint: limit lower=-3.1415 upper=3.1415 effort=1 velocity=1 -> lower=-3.1415 upper=3.1415 effort=1.5 velocity=59
- joint right_elbow_powered_joint: limit lower=-3.1415 upper=3.1415 effort=1 velocity=1 -> lower=-3.1415 upper=3.1415 effort=1.5 velocity=59
- joint right_hip_pitch_powered_joint: limit lower=-3.1415 upper=3.1415 effort=1 velocity=1 -> lower=-3.1415 upper=3.1415 effort=1.5 velocity=59
- joint right_hip_roll_powered_joint: limit lower=-3.1415 upper=3.1415 effort=1 velocity=1 -> lower=-3.1415 upper=3.1415 effort=1.5 velocity=59
- joint right_hip_yaw_powered_joint: limit lower=-3.1415 upper=3.1415 effort=1 velocity=1 -> lower=-3.1415 upper=3.1415 effort=1.5 velocity=59
- joint right_knee_pitch_powered_joint: limit lower=-3.1415 upper=3.1415 effort=1 velocity=1 -> lower=-3.1415 upper=3.1415 effort=1.5 velocity=59
- joint right_shoulder_pitch_powered_joint: limit lower=-3.1415 upper=3.1415 effort=1 velocity=1 -> lower=-3.1415 upper=3.1415 effort=1.5 velocity=59
- joint right_shoulder_roll_powered_joint: limit lower=-3.1415 upper=3.1415 effort=1 velocity=1 -> lower=-3.1415 upper=3.1415 effort=1.5 velocity=59

File: hros1_description/urdf/hros1_robot.urdf.xacro (robot description, xacro)
@@ -1,4 +1,5 @@
 <?xml version="1.0"?>
 <robot name="hros1" xmlns:xacro="http://www.ros.org/wiki/xacro">
+    <xacro:include filename="$(find hros1_description)/urdf/hros1_common.xacro"/>
     <xacro:include filename="$(find hros1_description)/urdf/hros1_dimensions.xacro"/>
     <xacro:include filename="$(find hros1_description)/urdf/hros1_body.xacro"/>
@@ -8,4 +9,5 @@
     <xacro:include filename="$(find hros1_description)/urdf/hros1_right_arm.xacro"/>
     <xacro:include filename="$(find hros1_description)/urdf/hros1_right_leg.xacro"/>
+    <xacro:include filename="$(find hros1_description)/urdf/hros1_transmission.xacro"/>
     <xacro:body_links />
     <xacro:body_joints />
@@ -20,6 +22,7 @@
     <xacro:right_leg_links />
     <xacro:right_leg_joints />
+    <xacro:hros1_transmissions/>
     <link name="world"/>
-    <joint name="fixed_joint" type="free">
+    <joint name="fixed_joint" type="floating">
         <parent link="world"/>
         <child link="body_structure_link"/>
